File: Week3IntoKiCAD/CHARLIE/CHARLIE.kicad_pcb (KiCad board)
At the start: 2 copper layers, 37 x 11 mm, 12 parts

Commit message: Week 3 charlie routing underway
Parts:
- added J1: Conn_01x04_Male, Connector_PinHeader_2.54mm:PinHeader_1x04_P2.54mm_Vertical, F.Cu at (202.8, 100.1)
- added R1: R, Resistor_SMD:R_0603_1608Metric, F.Cu at (186.4, 101.3)
- added R2: R, Resistor_SMD:R_0603_1608Metric, F.Cu at (186.4, 104.3)
- added R3: R, Resistor_SMD:R_0603_1608Metric, F.Cu at (186.4, 106.3)
- added R4: R, Resistor_SMD:R_0603_1608Metric, F.Cu at (186.4, 108.3)
Routing:
- net /IO1: track 0.00 -> 54.8 mm, vias 0 -> 5
- net /IO3: track 0.00 -> 36.8 mm, vias 0 -> 2
- net /IO2: track 0.00 -> 30.8 mm, vias 0 -> 2
- net /IO4: track 0.00 -> 29.2 mm, vias 0 -> 3
Other:
- board size 37 x 11 mm -> 40 x 11 mm
- net class Default Gee added: clearance 0.2032, trace_width 0.2032, via_dia 0.8, via_drill 0.4
