File: Week3IntoKiCAD/CHARLIE/CHARLIE.kicad_pcb (KiCad board)
At the start: 2 copper layers, 40 x 11 mm, 17 parts

Commit message: Had forgot to save OPPPs resync
Parts:
- added G***: LOGO, CHARLIE:topsilk, F.Cu at (172.4, 104.8)

Commit message: Week 3 Complete
Parts:
- added G***: LOGO, CHARLIE:bottomsilk, B.Cu at (169.4, 105.3)
