File: Week4BUBBLEWATCH/BubbleWatch.sch (KiCad schematic (older format))
At the start: 13 parts, among them U1 RedRetroBubbleDisplay, U2 RedRetroBubbleDisplay, U3 STM32F030C8Tx

Commit message: Schematic done datasheet added
Parts:
- removed R?: R, symbol Device:R
- added C1: 4.7uF, Capacitors_SMD:C_0603, symbol Device:C
- added C2, C3, C6, C7: 100nF, Capacitors_SMD:C_0603, symbol Device:C
- added C5: 1uF, Capacitors_SMD:C_0603, symbol Device:C
- added J1, J2: Conn_02x02_Counter_Clockwise, Pin_Headers:Pin_Header_Straight_2x02_Pitch2.54mm_SMD, symbol Conn_02x02_Counter_Clockwise
- added J3: Conn_01x05, Pin_Headers:Pin_Header_Straight_1x05_Pitch2.54mm, symbol Conn_01x05
- added R2: 200k, Resistors_SMD:R_0603, symbol Device:R
- added R3: 10k, Resistors_SMD:R_0603, symbol Device:R
- added SW1, SW2, SW3, SW4: SW_Push, Buttons_Switches_SMD:SW_SPST_B3U-3000P-B, symbol SW_Push
- added Y1: Crystal, Crystals:Crystal_DS10_d1.0mm_l4.3mm_Horizontal, symbol Crystal
- BT1, BT2: footprint (none) -> Battery_Holders:Keystone_3000_1x12mm-CoinCell
- C4: renamed from C?; value C -> 10nF; footprint (none) -> Capacitors_SMD:C_0603
- C8: renamed from C?; value C -> 4.7uF; footprint (none) -> Capacitors_SMD:C_0603
- L1: renamed from L?; value L -> 4.7uH; footprint (none) -> Inductors_SMD:L_Taiyo-Yuden_NR-30xx
- R1: renamed from R?; value R -> 330K; footprint (none) -> Resistors_SMD:R_0603
- RN1, RN2: renamed from RN?; value R_Pack04 -> 220R; footprint (none) -> Resistors_SMD:R_Array_Concave_4x0402
- U1, U2: footprint (none) -> Housings_DIP:DIP-12_W7.62mm_Socket_LongPads
- gave numbers to parts that had none: 1
Connections:
- net labels added: +3.3v, BATMON1, BATMON2, BUTTON1, BUTTON2, BUTTON3, BUTTON4, SWDCLK, SWDIO, VDD, VDDA, VSS, VSSA
- net labels removed: +5V
- wire segments 72 -> 163
Other:
- note added: "Decoupleing"
- note added: "Programming header"
- note added: "Top/Bottom Board interconnect"
