File: Week4BUBBLEWATCH/BubbleWatch.sch (KiCad schematic (older format))
At the start: 29 parts, among them J1 Conn_02x02_Counter_Clockwise, J2 Conn_02x02_Counter_Clockwise, J3 Conn_01x05, SW1 SW_Push, SW2 SW_Push, SW3 SW_Push, SW4 SW_Push, U1 RedRetroBubbleDisplay, U2 RedRetroBubbleDisplay, U3 STM32F030C8Tx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

Commit message: recommited to update project files for kicad
Parts:
- BT1, BT2: footprint Battery_Holders:Keystone_3000_1x12mm-CoinCell -> Battery:BatteryHolder_Keystone_3000_1x12mm
- C1, C2, C3, C4, C5, C6, C7, C8, C9: footprint Capacitors_SMD:C_0603 -> Capacitor_SMD:C_0603_1608Metric
- J1, J2: footprint Pin_Headers:Pin_Header_Straight_2x02_Pitch2.54mm_SMD -> Connector_PinHeader_2.54mm:PinHeader_2x02_P2.54mm_Vertical
- J3: footprint Pin_Headers:Pin_Header_Straight_1x05_Pitch2.54mm -> Connector_Harwin:Harwin_M20-89005xx_1x05_P2.54mm_Horizontal
- L1: footprint Inductors_SMD:L_Taiyo-Yuden_NR-30xx -> Inductor_SMD:L_Taiyo-Yuden_NR-30xx
- R1, R2, R3: footprint Resistors_SMD:R_0603 -> Resistor_SMD:R_0603_1608Metric
- RN1, RN2: footprint Resistors_SMD:R_Array_Concave_4x0402 -> Resistor_SMD:R_Array_Concave_4x0402
- SW1, SW2, SW3, SW4: footprint Buttons_Switches_SMD:SW_SPST_B3U-3000P-B -> Button_Switch_SMD:Panasonic_EVQPUM_EVQPUD
- U1, U2: footprint Housings_DIP:DIP-12_W7.62mm_Socket_LongPads -> Package_DIP:DIP-12_W7.62mm_Socket
- U4: footprint TO_SOT_Packages_SMD:SOT-23-6 -> Package_TO_SOT_SMD:SOT-23-6
- Y1: footprint Crystals:Crystal_DS10_d1.0mm_l4.3mm_Horizontal -> Crystal:Crystal_DS10_D1.0mm_L4.3mm_Horizontal_1EP_style1
Changed lines of the file:
@@
 F 0 "U1" H 4750 4217 60  0000 C CNN
 F 1 "RedRetroBubbleDisplay" H 4750 4096 80  0000 C CNB
-F 2 "Housings_DIP:DIP-12_W7.62mm_Socket_LongPads" H 4800 4100 60  0001 C CNN
+F 2 "Package_DIP:DIP-12_W7.62mm_Socket" H 4800 4100 60  0001 C CNN
 F 3 "" H 4800 4100 60  0001 C CNN
 	1    4750 3550
@@
 F 0 "U2" H 4750 5467 60  0000 C CNN
 F 1 "RedRetroBubbleDisplay" H 4750 5346 80  0000 C CNB
-F 2 "Housings_DIP:DIP-12_W7.62mm_Socket_LongPads" H 4800 5350 60  0001 C CNN
+F 2 "Package_DIP:DIP-12_W7.62mm_Socket" H 4800 5350 60  0001 C CNN
 F 3 "" H 4800 5350 60  0001 C CNN
 	1    4750 4800
@@
 F 0 "RN1" H 8388 3846 50  0000 L CNN
 F 1 "220R" H 8388 3755 50  0000 L CNN
-F 2 "Resistors_SMD:R_Array_Concave_4x0402" V 8475 3800 50  0001 C CNN
+F 2 "Resistor_SMD:R_Array_Concave_4x0402" V 8475 3800 50  0001 C CNN
 F 3 "~" H 8200 3800 50  0001 C CNN
 	1    8200 3800
@@
 F 0 "C4" H 3865 6596 50  0000 L CNN
 F 1 "10nF" H 3865 6505 50  0000 L CNN
-F 2 "Capacitors_SMD:C_0603" H 3788 6400 50  0001 C CNN
+F 2 "Capacitor_SMD:C_0603_1608Metric" H 3788 6400 50  0001 C CNN
 F 3 "~" H 3750 6550 50  0001 C CNN
 	1    3750 6550
@@
 F 0 "RN2" H 8388 4696 50  0000 L CNN
 F 1 "220R" H 8388 4605 50  0000 L CNN
-F 2 "Resistors_SMD:R_Array_Concave_4x0402" V 8475 4650 50  0001 C CNN
+F 2 "Resistor_SMD:R_Array_Concave_4x0402" V 8475 4650 50  0001 C CNN
 F 3 "~" H 8200 4650 50  0001 C CNN
 	1    8200 4650
@@
 F 0 "U4" H 9550 2267 50  0000 C CNN
 F 1 "MCP1640BCH" H 9550 2176 50  0000 C CNN
-F 2 "TO_SOT_Packages_SMD:SOT-23-6" H 9600 1550 50  0001 L CIN
+F 2 "Package_TO_SOT_SMD:SOT-23-6" H 9600 1550 50  0001 L CIN
 F 3 "http://ww1.microchip.com/downloads/en/DeviceDoc/20002234D.pdf" H 9300 2250 50  0001 C CNN
 	1    9550 1800
@@
 F 0 "L1" H 9653 1196 50  0000 L CNN
 F 1 "4.7uH" H 9653 1105 50  0000 L CNN
-F 2 "Inductors_SMD:L_Taiyo-Yuden_NR-30xx" H 9600 1150 50  0001 C CNN
+F 2 "Inductor_SMD:L_Taiyo-Yuden_NR-30xx" H 9600 1150 50  0001 C CNN
 F 3 "~" H 9600 1150 50  0001 C CNN
 	1    9600 1150
@@
 F 0 "R1" H 10320 2046 50  0000 L CNN
 F 1 "330K" H 10320 1955 50  0000 L CNN
-F 2 "Resistors_SMD:R_0603" V 10180 2000 50  0001 C CNN
+F 2 "Resistor_SMD:R_0603_1608Metric" V 10180 2000 50  0001 C CNN
 F 3 "~" H 10250 2000 50  0001 C CNN
 	1    10250 2000
@@
 F 0 "BT2" H 7118 1896 50  0000 L CNN
 F 1 "Battery_Cell" H 7118 1805 50  0000 L CNN
-F 2 "Battery_Holders:Keystone_3000_1x12mm-CoinCell" V 7000 1860 50  0001 C CNN
+F 2 "Battery:BatteryHolder_Keystone_3000_1x12mm" V 7000 1860 50  0001 C CNN
 F 3 "~" V 7000 1860 50  0001 C CNN
 	1    7000 1800
@@
 F 0 "BT1" H 6368 1896 50  0000 L CNN
 F 1 "Battery_Cell" H 6368 1805 50  0000 L CNN
-F 2 "Battery_Holders:Keystone_3000_1x12mm-CoinCell" V 6250 1860 50  0001 C CNN
+F 2 "Battery:BatteryHolder_Keystone_3000_1x12mm" V 6250 1860 50  0001 C CNN
 F 3 "~" V 6250 1860 50  0001 C CNN
 	1    6250 1800
@@
 F 0 "C5" H 4265 6596 50  0000 L CNN
 F 1 "1uF" H 4265 6505 50  0000 L CNN
-F 2 "Capacitors_SMD:C_0603" H 4188 6400 50  0001 C CNN
+F 2 "Capacitor_SMD:C_0603_1608Metric" H 4188 6400 50  0001 C CNN
 F 3 "~" H 4150 6550 50  0001 C CNN
 	1    4150 6550
@@
 F 0 "C1" H 5065 6546 50  0000 L CNN
 F 1 "4.7uF" H 5065 6455 50  0000 L CNN
-F 2 "Capacitors_SMD:C_0603" H 4988 6350 50  0001 C CNN
+F 2 "Capacitor_SMD:C_0603_1608Metric" H 4988 6350 50  0001 C CNN
 F 3 "~" H 4950 6500 50  0001 C CNN
 	1    4950 6500
@@
 F 0 "SW1" H 1750 1250 50  0000 L CNN
 F 1 "SW_Push" H 1700 1090 50  0000 C CNN
-F 2 "Buttons_Switches_SMD:SW_SPST_B3U-3000P-B" H 1700 1350 50  0001 C CNN
+F 2 "Button_Switch_SMD:Panasonic_EVQPUM_EVQPUD" H 1700 1350 50  0001 C CNN
 F 3 "" H 1700 1350 50  0001 C CNN
 	1    1700 1150
@@
 F 0 "SW2" H 1750 1600 50  0000 L CNN
 F 1 "SW_Push" H 1700 1440 50  0000 C CNN
-F 2 "Buttons_Switches_SMD:SW_SPST_B3U-3000P-B" H 1700 1700 50  0001 C CNN
+F 2 "Button_Switch_SMD:Panasonic_EVQPUM_EVQPUD" H 1700 1700 50  0001 C CNN
 F 3 "" H 1700 1700 50  0001 C CNN
 	1    1700 1500
@@
 F 0 "SW3" H 1750 1950 50  0000 L CNN
 F 1 "SW_Push" H 1700 1790 50  0000 C CNN
-F 2 "Buttons_Switches_SMD:SW_SPST_B3U-3000P-B" H 1700 2050 50  0001 C CNN
+F 2 "Button_Switch_SMD:Panasonic_EVQPUM_EVQPUD" H 1700 2050 50  0001 C CNN
 F 3 "" H 1700 2050 50  0001 C CNN
 	1    1700 1850
@@
 F 0 "SW4" H 1750 2300 50  0000 L CNN
 F 1 "SW_Push" H 1700 2140 50  0000 C CNN
-F 2 "Buttons_Switches_SMD:SW_SPST_B3U-3000P-B" H 1700 2400 50  0001 C CNN
+F 2 "Button_Switch_SMD:Panasonic_EVQPUM_EVQPUD" H 1700 2400 50  0001 C CNN
 F 3 "" H 1700 2400 50  0001 C CNN
 	1    1700 2200
@@
 F 0 "R2" H 10320 2446 50  0000 L CNN
 F 1 "200k" H 10320 2355 50  0000 L CNN
-F 2 "Resistors_SMD:R_0603" V 10180 2400 50  0001 C CNN
+F 2 "Resistor_SMD:R_0603_1608Metric" V 10180 2400 50  0001 C CNN
 F 3 "~" H 10250 2400 50  0001 C CNN
 	1    10250 2400
@@
 F 0 "J1" H 3800 1700 50  0000 C CNN
 F 1 "Conn_02x02_Counter_Clockwise" H 3800 1400 50  0000 C CNN
-F 2 "Pin_Headers:Pin_Header_Straight_2x02_Pitch2.54mm_SMD" H 3750 1600 50  0001 C CNN
+F 2 "Connector_PinHeader_2.54mm:PinHeader_2x02_P2.54mm_Vertical" H 3750 1600 50  0001 C CNN
 F 3 "" H 3750 1600 50  0001 C CNN
 	1    3750 1600
@@
 F 0 "J2" H 3800 2150 50  0000 C CNN
 F 1 "Conn_02x02_Counter_Clockwise" H 3800 1850 50  0000 C CNN
-F 2 "Pin_Headers:Pin_Header_Straight_2x02_Pitch2.54mm_SMD" H 3750 2050 50  0001 C CNN
+F 2 "Connector_PinHeader_2.54mm:PinHeader_2x02_P2.54mm_Vertical" H 3750 2050 50  0001 C CNN
 F 3 "" H 3750 2050 50  0001 C CNN
 	1    3750 2050
@@
 F 0 "J3" H 10200 4450 50  0000 C CNN
 F 1 "Conn_01x05" H 10200 3850 50  0000 C CNN
-F 2 "Pin_Headers:Pin_Header_Straight_1x05_Pitch2.54mm" H 10200 4150 50  0001 C CNN
+F 2 "Connector_Harwin:Harwin_M20-89005xx_1x05_P2.54mm_Horizontal" H 10200 4150 50  0001 C CNN
 F 3 "" H 10200 4150 50  0001 C CNN
 	1    10200 4150
@@
 F 0 "C2" H 5465 6546 50  0000 L CNN
 F 1 "100nF" H 5465 6455 50  0000 L CNN
-F 2 "Capacitors_SMD:C_0603" H 5388 6350 50  0001 C CNN
+F 2 "Capacitor_SMD:C_0603_1608Metric" H 5388 6350 50  0001 C CNN
 F 3 "~" H 5350 6500 50  0001 C CNN
 	1    5350 6500
@@
 F 0 "C3" H 5915 6546 50  0000 L CNN
 F 1 "100nF" H 5915 6455 50  0000 L CNN
-F 2 "Capacitors_SMD:C_0603" H 5838 6350 50  0001 C CNN
+F 2 "Capacitor_SMD:C_0603_1608Metric" H 5838 6350 50  0001 C CNN
 F 3 "~" H 5800 6500 50  0001 C CNN
 	1    5800 6500
@@
 F 0 "Y1" H 8850 5850 50  0000 C CNN
 F 1 "Crystal" H 8850 5550 50  0000 C CNN
-F 2 "Crystals:Crystal_DS10_d1.0mm_l4.3mm_Horizontal" H 8850 5700 50  0001 C CNN
+F 2 "Crystal:Crystal_DS10_D1.0mm_L4.3mm_Horizontal_1EP_style1" H 8850 5700 50  0001 C CNN
 F 3 "" H 8850 5700 50  0001 C CNN
 	1    8850 5700
@@
 F 0 "C6" H 8565 6096 50  0000 L CNN
 F 1 "12pF" H 8565 6005 50  0000 L CNN
-F 2 "Capacitors_SMD:C_0603" H 8488 5900 50  0001 C CNN
+F 2 "Capacitor_SMD:C_0603_1608Metric" H 8488 5900 50  0001 C CNN
 F 3 "~" H 8450 6050 50  0001 C CNN
 	1    8450 6050
@@
 F 0 "R3" H 7470 5846 50  0000 L CNN
 F 1 "10k" H 7470 5755 50  0000 L CNN
-F 2 "Resistors_SMD:R_0603" V 7330 5800 50  0001 C CNN
+F 2 "Resistor_SMD:R_0603_1608Metric" V 7330 5800 50  0001 C CNN
 F 3 "~" H 7400 5800 50  0001 C CNN
 	1    7400 5800
@@
 F 0 "C8" H 9315 6096 50  0000 L CNN
 F 1 "12pF" H 9315 6005 50  0000 L CNN
-F 2 "Capacitors_SMD:C_0603" H 9238 5900 50  0001 C CNN
+F 2 "Capacitor_SMD:C_0603_1608Metric" H 9238 5900 50  0001 C CNN
 F 3 "~" H 9200 6050 50  0001 C CNN
 	1    9200 6050
@@
 F 0 "C7" H 8715 2096 50  0000 L CNN
 F 1 "4.7uF" H 8715 2005 50  0000 L CNN
-F 2 "Capacitors_SMD:C_0603" H 8638 1900 50  0001 C CNN
+F 2 "Capacitor_SMD:C_0603_1608Metric" H 8638 1900 50  0001 C CNN
 F 3 "~" H 8600 2050 50  0001 C CNN
 	1    8600 2050
@@
 F 0 "C9" H 10815 2246 50  0000 L CNN
 F 1 "10uF" H 10815 2155 50  0000 L CNN
-F 2 "Capacitors_SMD:C_0603" H 10738 2050 50  0001 C CNN
+F 2 "Capacitor_SMD:C_0603_1608Metric" H 10738 2050 50  0001 C CNN
 F 3 "~" H 10700 2200 50  0001 C CNN
 	1    10700 2200

Commit message: more routing work
Connections:
- wire segments 194 -> 196
Changed lines of the file:
@@
 Connection ~ 4150 6950
 Wire Wire Line
-	4050 1600 4450 1600
-Wire Wire Line
 	4050 1700 4450 1700
 Wire Wire Line
@@
 Wire Wire Line
 	3550 1700 3100 1700
-Wire Wire Line
-	4050 2050 4450 2050
 Wire Wire Line
 	4050 2150 4450 2150
@@
 Wire Wire Line
 	10700 2350 10700 2700
+$Comp
+L power:+3.3V #PWR0102
+U 1 1 5B6A8117
+P 4550 1550
+F 0 "#PWR0102" H 4550 1400 50  0001 C CNN
+F 1 "+3.3V" H 4565 1723 50  0000 C CNN
+F 2 "" H 4550 1550 50  0001 C CNN
+F 3 "" H 4550 1550 50  0001 C CNN
+	1    4550 1550
+	1    0    0    -1
+$EndComp
+$Comp
+L power:+3.3V #PWR0103
+U 1 1 5B6A815C
+P 4550 2000
+F 0 "#PWR0103" H 4550 1850 50  0001 C CNN
+F 1 "+3.3V" H 4565 2173 50  0000 C CNN
+F 2 "" H 4550 2000 50  0001 C CNN
+F 3 "" H 4550 2000 50  0001 C CNN
+	1    4550 2000
+	1    0    0    -1
+$EndComp
+Wire Wire Line
+	4550 2050 4550 2000
+Wire Wire Line
+	4050 2050 4550 2050
+Wire Wire Line
+	4550 1600 4550 1550
+Wire Wire Line
+	4050 1600 4550 1600
 $EndSCHEMATC

Commit message: More work on week 4
Converting display placements to SMT to allow mor room on board.
Parts:
- J1, J2: footprint Connector_PinHeader_2.54mm:PinHeader_2x02_P2.54mm_Vertical -> Connector_PinHeader_2.54mm:PinHeader_2x02_P2.54mm_Vertical_SMD
- U1, U2: footprint Package_DIP:DIP-12_W7.62mm_Socket -> Package_DIP:DIP-12_W7.62mm_SMDSocket_SmallPads
Changed lines of the file:
@@
 F 0 "U1" H 4750 4217 60  0000 C CNN
 F 1 "RedRetroBubbleDisplay" H 4750 4096 80  0000 C CNB
-F 2 "Package_DIP:DIP-12_W7.62mm_Socket" H 4800 4100 60  0001 C CNN
+F 2 "Package_DIP:DIP-12_W7.62mm_SMDSocket_SmallPads" H 4800 4100 60  0001 C CNN
 F 3 "" H 4800 4100 60  0001 C CNN
 	1    4750 3550
@@
 F 0 "U2" H 4750 5467 60  0000 C CNN
 F 1 "RedRetroBubbleDisplay" H 4750 5346 80  0000 C CNB
-F 2 "Package_DIP:DIP-12_W7.62mm_Socket" H 4800 5350 60  0001 C CNN
+F 2 "Package_DIP:DIP-12_W7.62mm_SMDSocket_SmallPads" H 4800 5350 60  0001 C CNN
 F 3 "" H 4800 5350 60  0001 C CNN
 	1    4750 4800
@@
 F 0 "J1" H 3800 1700 50  0000 C CNN
 F 1 "Conn_02x02_Counter_Clockwise" H 3800 1400 50  0000 C CNN
-F 2 "Connector_PinHeader_2.54mm:PinHeader_2x02_P2.54mm_Vertical" H 3750 1600 50  0001 C CNN
+F 2 "Connector_PinHeader_2.54mm:PinHeader_2x02_P2.54mm_Vertical_SMD" H 3750 1600 50  0001 C CNN
 F 3 "" H 3750 1600 50  0001 C CNN
 	1    3750 1600
@@
 F 0 "J2" H 3800 2150 50  0000 C CNN
 F 1 "Conn_02x02_Counter_Clockwise" H 3800 1850 50  0000 C CNN
-F 2 "Connector_PinHeader_2.54mm:PinHeader_2x02_P2.54mm_Vertical" H 3750 2050 50  0001 C CNN
+F 2 "Connector_PinHeader_2.54mm:PinHeader_2x02_P2.54mm_Vertical_SMD" H 3750 2050 50  0001 C CNN
 F 3 "" H 3750 2050 50  0001 C CNN
 	1    3750 2050
