File: Week4BUBBLEWATCH/BubbleWatch.sch (KiCad schematic (older format))
At the start: 29 parts, among them J1 Conn_02x02_Counter_Clockwise, J2 Conn_02x02_Counter_Clockwise, J3 Conn_01x05, SW1 SW_Push, SW2 SW_Push, SW3 SW_Push, SW4 SW_Push, U1 RedRetroBubbleDisplay, U2 RedRetroBubbleDisplay, U3 STM32F030C8Tx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

Commit message: repush schmatic
Parts:
- U1, U2: footprint Package_DIP:DIP-12_W7.62mm_SMDSocket_SmallPads -> Week4BUBBLEWATCH:DIP-12_W7.62mm_SMDSocket_SmallPads
Changed lines of the file:
@@
 F 0 "U1" H 4750 4217 60  0000 C CNN
 F 1 "RedRetroBubbleDisplay" H 4750 4096 80  0000 C CNB
-F 2 "Package_DIP:DIP-12_W7.62mm_SMDSocket_SmallPads" H 4800 4100 60  0001 C CNN
+F 2 "Week4BUBBLEWATCH:DIP-12_W7.62mm_SMDSocket_SmallPads" H 4800 4100 60  0001 C CNN
 F 3 "" H 4800 4100 60  0001 C CNN
 	1    4750 3550
@@
 F 0 "U2" H 4750 5467 60  0000 C CNN
 F 1 "RedRetroBubbleDisplay" H 4750 5346 80  0000 C CNB
-F 2 "Package_DIP:DIP-12_W7.62mm_SMDSocket_SmallPads" H 4800 5350 60  0001 C CNN
+F 2 "Week4BUBBLEWATCH:DIP-12_W7.62mm_SMDSocket_SmallPads" H 4800 5350 60  0001 C CNN
 F 3 "" H 4800 5350 60  0001 C CNN
 	1    4750 4800
