File: Week4BUBBLEWATCH/BubbleWatch.kicad_pcb (KiCad board)
At the start: 2 copper layers, 79 x 36 mm, 37 parts, among them J1 Conn_02x02_Counter_Clockwise, J2 Conn_02x02_Counter_Clockwise, J3 Conn_01x05, SW1 SW_Push, SW2 SW_Push, SW3 SW_Push, SW4 SW_Push, U1 RedRetroBubbleDisplay, U2 RedRetroBubbleDisplay, U3 STM32F030C8Tx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

Commit message: end of day commit
Parts:
- C6, C8: moved to F.Cu
- moved J3 84.6 mm to (144.0, 95.0)
- moved C8 84.1 mm to (141.0, 74.0), turned to 180 degrees
- moved Y1 69.6 mm to (142.0, 77.0)
- moved C6 6.96 mm to (141.2, 79.0), turned to 180 degrees
- moved SW1 6.69 mm to (158.0, 65.0)
Other:
- board size 79 x 36 mm -> 84 x 36 mm
Changed lines of the file:
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@@
   )
   (module Crystal:Crystal_DS10_D1.0mm_L4.3mm_Horizontal_1EP_style1 (layer F.Cu)
-    (at 210.9 86.8 90)
+    (at 142 77 90)
     (descr "Crystal THT DS10 4.3mm length 1.0mm diameter http://www.microcrystal.com/images/_Product-Documentation/03_TF_metal_Packages/01_Datasheet/DS-Series.pdf")
     (tags ['DS10'])
@@
   )
   (module Buttons_Switches_SMD:SW_SPST_B3U-3000P (layer B.Cu)
-    (at 163.5 61.2 90)
+    (at 158 65 90)
     (descr "Ultra-small-sized Tactile Switch with High Contact Reliability, Side-actuated Model, without Ground Terminal, without Boss")
     (tags "Tactile Switch")
@@
   )
   (module Connector_Harwin:Harwin_M20-89005xx_1x05_P2.54mm_Horizontal (layer F.Cu)
-    (at 227 78.6 90)
+    (at 144 95 90)
     (descr "Harwin Male Horizontal Surface Mount Single Row 2.54mm (0.1 inch) Pitch PCB Connector, M20-89005xx, 5 Pins per row (https://cdn.harwin.com/pdfs/M20-890.pdf), generated with kicad-footprint-generator")
     (tags "connector Harwin M20-890 horizontal")
@@
     )
   )
-  (module Capacitor_SMD:C_0603_1608Metric (layer B.Cu)
-    (at 143.1 85.7 135)
+  (module Capacitor_SMD:C_0603_1608Metric (layer F.Cu)
+    (at 141.212499 79 180)
     (descr "Capacitor SMD 0603 (1608 Metric), square (rectangular) end terminal, IPC_7351 nominal, (Body size source: http://www.tortai-tech.com/upload/download/2011102023233369053.pdf), generated with kicad-footprint-generator")
     (tags capacitor)
     (attr smd)
-    (fp_text reference C6 (at 0 1.43 135) (layer B.SilkS)
-      (effects (font (size 1 1) (thickness 0.15)) (justify mirror))
-    )
-    (fp_text value 12pF (at 0 -1.43 135) (layer B.Fab)
-      (effects (font (size 1 1) (thickness 0.15)) (justify mirror))
-    )
-    (fp_line (start -0.8 -0.4) (end -0.8 0.4) (layer B.Fab) (width 0.1))
-    (fp_line (start -0.8 0.4) (end 0.8 0.4) (layer B.Fab) (width 0.1))
-    (fp_line (start 0.8 0.4) (end 0.8 -0.4) (layer B.Fab) (width 0.1))
-    (fp_line (start 0.8 -0.4) (end -0.8 -0.4) (layer B.Fab) (width 0.1))
-    (fp_line (start -0.162779 0.51) (end 0.162779 0.51) (layer B.SilkS) (width 0.12))
-    (fp_line (start -0.162779 -0.51) (end 0.162779 -0.51) (layer B.SilkS) (width 0.12))
-    (fp_line (start -1.48 -0.73) (end -1.48 0.73) (layer B.CrtYd) (width 0.05))
-    (fp_line (start -1.48 0.73) (end 1.48 0.73) (layer B.CrtYd) (width 0.05))
-    (fp_line (start 1.48 0.73) (end 1.48 -0.73) (layer B.CrtYd) (width 0.05))
-    (fp_line (start 1.48 -0.73) (end -1.48 -0.73) (layer B.CrtYd) (width 0.05))
-    (fp_text user %R (at 0 0 135) (layer B.Fab)
-      (effects (font (size 0.4 0.4) (thickness 0.06)) (justify mirror))
-    )
-    (pad 1 smd roundrect (at -0.787501 0 135) (size 0.875 0.95) (layers B.Cu B.Paste B.Mask) (roundrect_rratio 0.25)
+    (fp_text reference C6 (at 0 -1.43 180) (layer F.SilkS)
+      (effects (font (size 1 1) (thickness 0.15)))
+    )
+    (fp_text value 12pF (at 0 1.43 180) (layer F.Fab)
+      (effects (font (size 1 1) (thickness 0.15)))
+    )
+    (fp_line (start -0.8 0.4) (end -0.8 -0.4) (layer F.Fab) (width 0.1))
+    (fp_line (start -0.8 -0.4) (end 0.8 -0.4) (layer F.Fab) (width 0.1))
+    (fp_line (start 0.8 -0.4) (end 0.8 0.4) (layer F.Fab) (width 0.1))
+    (fp_line (start 0.8 0.4) (end -0.8 0.4) (layer F.Fab) (width 0.1))
+    (fp_line (start -0.162779 -0.51) (end 0.162779 -0.51) (layer F.SilkS) (width 0.12))
+    (fp_line (start -0.162779 0.51) (end 0.162779 0.51) (layer F.SilkS) (width 0.12))
+    (fp_line (start -1.48 0.73) (end -1.48 -0.73) (layer F.CrtYd) (width 0.05))
+    (fp_line (start -1.48 -0.73) (end 1.48 -0.73) (layer F.CrtYd) (width 0.05))
+    (fp_line (start 1.48 -0.73) (end 1.48 0.73) (layer F.CrtYd) (width 0.05))
+    (fp_line (start 1.48 0.73) (end -1.48 0.73) (layer F.CrtYd) (width 0.05))
+    (fp_text user %R (at 0 0 180) (layer F.Fab)
+      (effects (font (size 0.4 0.4) (thickness 0.06)))
+    )
+    (pad 1 smd roundrect (at -0.787501 0 180) (size 0.875 0.95) (layers F.Cu F.Paste F.Mask) (roundrect_rratio 0.25)
       (net 4 /RTC_XTAL_IN))
-    (pad 2 smd roundrect (at 0.787501 0 135) (size 0.875 0.95) (layers B.Cu B.Paste B.Mask) (roundrect_rratio 0.25)
+    (pad 2 smd roundrect (at 0.787501 0 180) (size 0.875 0.95) (layers F.Cu F.Paste F.Mask) (roundrect_rratio 0.25)
       (net 1 GND))
     (model ${KISYS3DMOD}/Capacitor_SMD.3dshapes/C_0603_1608Metric.wrl
@@
     )
   )
-  (module Capacitor_SMD:C_0603_1608Metric (layer B.Cu)
-    (at 221.143153 99.643153 315)
+  (module Capacitor_SMD:C_0603_1608Metric (layer F.Cu)
+    (at 141 74 180)
     (descr "Capacitor SMD 0603 (1608 Metric), square (rectangular) end terminal, IPC_7351 nominal, (Body size source: http://www.tortai-tech.com/upload/download/2011102023233369053.pdf), generated with kicad-footprint-generator")
     (tags capacitor)
     (attr smd)
-    (fp_text reference C8 (at 0 1.43 315) (layer B.SilkS)
-      (effects (font (size 1 1) (thickness 0.15)) (justify mirror))
-    )
-    (fp_text value 12pF (at 0 -1.43 315) (layer B.Fab)
-      (effects (font (size 1 1) (thickness 0.15)) (justify mirror))
-    )
-    (fp_text user %R (at 0 0 315) (layer B.Fab)
-      (effects (font (size 0.4 0.4) (thickness 0.06)) (justify mirror))
-    )
-    (fp_line (start 1.48 -0.73) (end -1.48 -0.73) (layer B.CrtYd) (width 0.05))
-    (fp_line (start 1.48 0.73) (end 1.48 -0.73) (layer B.CrtYd) (width 0.05))
-    (fp_line (start -1.48 0.73) (end 1.48 0.73) (layer B.CrtYd) (width 0.05))
-    (fp_line (start -1.48 -0.73) (end -1.48 0.73) (layer B.CrtYd) (width 0.05))
-    (fp_line (start -0.162779 -0.51) (end 0.162779 -0.51) (layer B.SilkS) (width 0.12))
-    (fp_line (start -0.162779 0.51) (end 0.162779 0.51) (layer B.SilkS) (width 0.12))
-    (fp_line (start 0.8 -0.4) (end -0.8 -0.4) (layer B.Fab) (width 0.1))
-    (fp_line (start 0.8 0.4) (end 0.8 -0.4) (layer B.Fab) (width 0.1))
-    (fp_line (start -0.8 0.4) (end 0.8 0.4) (layer B.Fab) (width 0.1))
-    (fp_line (start -0.8 -0.4) (end -0.8 0.4) (layer B.Fab) (width 0.1))
-    (pad 2 smd roundrect (at 0.787501 0 315) (size 0.875 0.95) (layers B.Cu B.Paste B.Mask) (roundrect_rratio 0.25)
-      (net 1 GND))
-    (pad 1 smd roundrect (at -0.787501 0 315) (size 0.875 0.95) (layers B.Cu B.Paste B.Mask) (roundrect_rratio 0.25)
+    (fp_text reference C8 (at 0 -1.43 180) (layer F.SilkS)
+      (effects (font (size 1 1) (thickness 0.15)))
+    )
+    (fp_text value 12pF (at 0 1.43 180) (layer F.Fab)
+      (effects (font (size 1 1) (thickness 0.15)))
+    )
+    (fp_text user %R (at 0 0 180) (layer F.Fab)
+      (effects (font (size 0.4 0.4) (thickness 0.06)))
+    )
+    (fp_line (start 1.48 0.73) (end -1.48 0.73) (layer F.CrtYd) (width 0.05))
+    (fp_line (start 1.48 -0.73) (end 1.48 0.73) (layer F.CrtYd) (width 0.05))
+    (fp_line (start -1.48 -0.73) (end 1.48 -0.73) (layer F.CrtYd) (width 0.05))
+    (fp_line (start -1.48 0.73) (end -1.48 -0.73) (layer F.CrtYd) (width 0.05))
+    (fp_line (start -0.162779 0.51) (end 0.162779 0.51) (layer F.SilkS) (width 0.12))
+    (fp_line (start -0.162779 -0.51) (end 0.162779 -0.51) (layer F.SilkS) (width 0.12))
+    (fp_line (start 0.8 0.4) (end -0.8 0.4) (layer F.Fab) (width 0.1))
+    (fp_line (start 0.8 -0.4) (end 0.8 0.4) (layer F.Fab) (width 0.1))
+    (fp_line (start -0.8 -0.4) (end 0.8 -0.4) (layer F.Fab) (width 0.1))
+    (fp_line (start -0.8 0.4) (end -0.8 -0.4) (layer F.Fab) (width 0.1))
+    (pad 2 smd roundrect (at 0.787501 0 180) (size 0.875 0.95) (layers F.Cu F.Paste F.Mask) (roundrect_rratio 0.25)
+      (net 1 GND))
+    (pad 1 smd roundrect (at -0.787501 0 180) (size 0.875 0.95) (layers F.Cu F.Paste F.Mask) (roundrect_rratio 0.25)
       (net 5 /RTC_XTAL_OUT))
     (model ${KISYS3DMOD}/Capacitor_SMD.3dshapes/C_0603_1608Metric.wrl
@@
     )
   )
-  (gr_arc (start 153 63) (end 155 63) (angle -90) (layer Edge.Cuts) (width 0.15))
-  (gr_arc (start 153 95) (end 153 97) (angle -90) (layer Edge.Cuts) (width 0.15))
-  (gr_arc (start 132 95) (end 130 95) (angle -90) (layer Edge.Cuts) (width 0.15))
-  (gr_arc (start 132 63) (end 132 61) (angle -90) (layer Edge.Cuts) (width 0.15))
-  (gr_line (start 153 61) (end 132 61) (layer Edge.Cuts) (width 0.15))
-  (gr_line (start 132 97) (end 153 97) (layer Edge.Cuts) (width 0.15))
-  (gr_line (start 130 63) (end 130 95) (layer Edge.Cuts) (width 0.15))
-  (gr_line (start 155 63) (end 155 95) (layer Edge.Cuts) (width 0.15))
+  (gr_arc (start 158 63) (end 160 63) (angle -90) (layer Edge.Cuts) (width 0.15))
+  (gr_arc (start 158 95) (end 158 97) (angle -90) (layer Edge.Cuts) (width 0.15))
+  (gr_arc (start 129 95) (end 127 95) (angle -90) (layer Edge.Cuts) (width 0.15))
+  (gr_arc (start 129 63) (end 129 61) (angle -90) (layer Edge.Cuts) (width 0.15))
+  (gr_line (start 158 61) (end 132 61) (layer Edge.Cuts) (width 0.15))
+  (gr_line (start 129 97) (end 158 97) (layer Edge.Cuts) (width 0.15))
+  (gr_line (start 127 63) (end 127 95) (layer Edge.Cuts) (width 0.15))
+  (gr_line (start 160 63) (end 160 95) (layer Edge.Cuts) (width 0.15))
   (gr_arc (start 115 88) (end 115 89) (angle -90) (layer Edge.Cuts) (width 0.15))
   (gr_line (start 116 88) (end 116 75) (layer Edge.Cuts) (width 0.15))
@@
   (gr_line (start 78 87) (end 78 71) (layer Edge.Cuts) (width 0.15))
   (gr_line (start 80 71) (end 80 87) (layer Edge.Cuts) (width 0.15))
-  (via (at 147 83.5) (size 0.8) (drill 0.4) (layers F.Cu B.Cu) (net 31))
   (segment (start 105 71.1) (end 97.695 71.1) (width 1) (layer F.Cu) (net 2) (status 30))
   (segment (start 97.695 71.1) (end 97.27 71.525) (width 1) (layer F.Cu) (net 2) (status 30))
@@
   (segment (start 149.65 85) (end 149.65 85.4532) (width 0.2032) (layer B.Cu) (net 25))
   (segment (start 149.65 85.4532) (end 150.201601 86.004801) (width 0.2032) (layer B.Cu) (net 25))
+  (via (at 147 83.5) (size 0.8) (drill 0.4) (layers F.Cu B.Cu) (net 31))
   (segment (start 130.7932 63.75) (end 132.0432 65) (width 0.2032) (layer F.Cu) (net 31))
   (segment (start 129.79 63.75) (end 130.7932 63.75) (width 0.2032) (layer F.Cu) (net 31))
