File: Week5LetsTryANewIC/Week5LetsTryANewIC.kicad_pcb (KiCad board)
At the start: 2 copper layers, 17 x 28 mm, 10 parts, among them J1 Conn_01x09_Male, U1 BMA400

Commit message: finished board updated readme
Parts:
- added G***: LOGO, ArtWorkAndSilks:topsilk, F.Cu at (162.5, 77.0)
- added G***: LOGO, ArtWorkAndSilks:bottomsilk, B.Cu at (162.0, 77.5)
