File: Week6BlinkALED/Blinkblock.sch (KiCad schematic (older format))
At the start: 18 parts, among them Q1 Q_Photo_NPN, Q2 Q_Photo_NPN, Q3 Q_Photo_NPN, U1 ATtiny10-TS

Commit message: Added gerbers to week 5
Other:
- note added: "Blinky LED"
- note added: "IR Comms"
- note added: "MCU and Programming"
- note added: "Power"
- moved on the sheet: U1
