File: Week7Theflower/THEFLOWER.kicad_pcb (KiCad board)
At the start: 2 copper layers, 37.3 x 37.3 mm, 1 part

Commit message: trying to make component choices work
Parts:
- added BT1: Battery_Cell, Battery:BatteryHolder_MPD_BC2003_1x2032, B.Cu at (157.2, 95.8)
- added C1: 1uF, Capacitor_SMD:C_0603_1608Metric, F.Cu at (195.8, 102.3)
- added C2: 100nF, Capacitor_SMD:C_0603_1608Metric, F.Cu at (211.8, 91.1)
- added D1: LED, LED_SMD:LED_0603_1608Metric, F.Cu at (177.5, 102.3)
- added D10: LED_RGB, LED_SMD:LED_RGB_5050-6, F.Cu at (206.6, 100.4)
- added D2: LED, LED_SMD:LED_0603_1608Metric, F.Cu at (180.6, 102.3)
- added D3: LED, LED_SMD:LED_0603_1608Metric, F.Cu at (183.6, 102.3)
- added D4: LED, LED_SMD:LED_0603_1608Metric, F.Cu at (186.7, 102.3)
- added D5: LED, LED_SMD:LED_0603_1608Metric, F.Cu at (189.7, 102.3)
- added D6: LED, LED_SMD:LED_0603_1608Metric, F.Cu at (192.8, 102.3)
- added D7: LED_RGB, LED_SMD:LED_RGB_5050-6, F.Cu at (206.6, 83.8)
- added D8: LED_RGB, LED_SMD:LED_RGB_5050-6, F.Cu at (206.6, 89.3)
- added D9: LED_RGB, LED_SMD:LED_RGB_5050-6, F.Cu at (206.6, 94.9)
- added R1: 3k3, Resistor_SMD:R_0603_1608Metric, F.Cu at (198.8, 102.3)
- added U1: LPC1104UK, Package_CSP:WLCSP-16_4x4_B2.17x2.32mm_P0.5mm, F.Cu at (157.0, 96.0)
- added U2: SN3218, Package_DFN_QFN:QFN-24_4x4mm_P0.5mm, B.Cu at (157.0, 111.0)

Commit message: more work on flower
Parts:
- moved D5 43.2 mm to (147.0, 96.0)
- moved D4 42.7 mm to (147.2, 86.0)
- moved D1 31.7 mm to (146.2, 106.8), turned to 45 degrees
- moved D6 26.6 mm to (167.0, 96.0)
- moved D3 23.3 mm to (166.8, 86.2)
- moved C1 17.7 mm to (179.6, 95.2)
- moved D2 13.9 mm to (167.2, 106.0)
- moved D7 3.18 mm to (206.6, 80.6)
Routing:
- net Net-(BT1-Pad2): vias 0 -> 2
Other:
- net class thin added: clearance 0.127, trace_width 0.127, via_dia 0.6, via_drill 0.3
- rule trace_min: 0.2 -> 0.125
- rule via_min_size: 0.4 -> 0.3
Changed lines of the file:
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@@
     (thickness 1.6)
     (drawings 8)
-    (tracks 0)
+    (tracks 2)
     (zones 0)
     (modules 17)
@@
   (page A4)
   (layers
-    (0 F.Cu signal hide)
+    (0 F.Cu signal)
     (31 B.Cu signal)
     (32 B.Adhes user hide)
@@
     (zone_clearance 0.508)
     (zone_45_only no)
-    (trace_min 0.2)
+    (trace_min 0.125)
     (segment_width 0.2)
     (edge_width 0.15)
     (via_size 0.8)
     (via_drill 0.4)
-    (via_min_size 0.4)
+    (via_min_size 0.3)
     (via_min_drill 0.3)
     (uvia_size 0.3)
@@
     (pad_to_mask_clearance 0.2)
     (aux_axis_origin 0 0)
-    (visible_elements 7FF9357F)
+    (visible_elements 7FF8B77F)
     (pcbplotparams
       (layerselection 0x010fc_ffffffff)
@@
     (uvia_dia 0.3)
     (uvia_drill 0.1)
+  )
+  (net_class thin ""
+    (clearance 0.127)
+    (trace_width 0.127)
+    (via_dia 0.6)
+    (via_drill 0.3)
+    (uvia_dia 0.3)
+    (uvia_drill 0.1)
     (add_net +3V3)
     (add_net /BACKLED1)
@@
   )
   (module Capacitor_SMD:C_0603_1608Metric (layer F.Cu)
-    (at 195.805001 102.295001)
+    (at 179.5875 95.2)
     (descr "Capacitor SMD 0603 (1608 Metric), square (rectangular) end terminal, IPC_7351 nominal, (Body size source: http://www.tortai-tech.com/upload/download/2011102023233369053.pdf), generated with kicad-footprint-generator")
     (tags capacitor)
@@
     (fp_line (start 1.48 -0.73) (end 1.48 0.73) (layer F.CrtYd) (width 0.05))
     (fp_line (start 1.48 0.73) (end -1.48 0.73) (layer F.CrtYd) (width 0.05))
-    (fp_text user %R (at 0 0) (layer F.Fab)
+    (fp_text user %R (at 0.0125 0) (layer F.Fab)
       (effects (font (size 0.4 0.4) (thickness 0.06)))
     )
@@
   )
   (module LED_SMD:LED_0603_1608Metric (layer F.Cu)
-    (at 177.545001 102.335001)
+    (at 146.2 106.8 45)
     (descr "LED SMD 0603 (1608 Metric), square (rectangular) end terminal, IPC_7351 nominal, (Body size source: http://www.tortai-tech.com/upload/download/2011102023233369053.pdf), generated with kicad-footprint-generator")
     (tags diode)
     (attr smd)
-    (fp_text reference D1 (at 0 -1.43) (layer F.SilkS)
+    (fp_text reference D1 (at 0 -1.43 45) (layer F.SilkS)
       (effects (font (size 1 1) (thickness 0.15)))
     )
-    (fp_text value LED (at 0 1.43) (layer F.Fab)
+    (fp_text value LED (at 0 1.43 45) (layer F.Fab)
       (effects (font (size 1 1) (thickness 0.15)))
     )
@@
     (fp_line (start 1.48 -0.73) (end 1.48 0.73) (layer F.CrtYd) (width 0.05))
     (fp_line (start 1.48 0.73) (end -1.48 0.73) (layer F.CrtYd) (width 0.05))
-    (fp_text user %R (at -1.545001 2.664999) (layer F.Fab)
+    (fp_text user %R (at -1.545001 2.664999 45) (layer F.Fab)
       (effects (font (size 0.4 0.4) (thickness 0.06)))
     )
-    (pad 1 smd roundrect (at -0.7875 0) (size 0.875 0.95) (layers F.Cu F.Paste F.Mask) (roundrect_rratio 0.25)
+    (pad 1 smd roundrect (at -0.7875 0 45) (size 0.875 0.95) (layers F.Cu F.Paste F.Mask) (roundrect_rratio 0.25)
       (net 5 /LEAF1))
-    (pad 2 smd roundrect (at 0.7875 0) (size 0.875 0.95) (layers F.Cu F.Paste F.Mask) (roundrect_rratio 0.25)
+    (pad 2 smd roundrect (at 0.7875 0 45) (size 0.875 0.95) (layers F.Cu F.Paste F.Mask) (roundrect_rratio 0.25)
       (net 3 +3V3))
     (model ${KISYS3DMOD}/LED_SMD.3dshapes/LED_0603_1608Metric.wrl
@@
   )
   (module LED_SMD:LED_0603_1608Metric (layer F.Cu)
-    (at 180.595001 102.335001)
+    (at 167.1875 106)
     (descr "LED SMD 0603 (1608 Metric), square (rectangular) end terminal, IPC_7351 nominal, (Body size source: http://www.tortai-tech.com/upload/download/2011102023233369053.pdf), generated with kicad-footprint-generator")
     (tags diode)
@@
   )
   (module LED_SMD:LED_0603_1608Metric (layer F.Cu)
-    (at 183.645001 102.335001)
+    (at 166.7875 86.2)
     (descr "LED SMD 0603 (1608 Metric), square (rectangular) end terminal, IPC_7351 nominal, (Body size source: http://www.tortai-tech.com/upload/download/2011102023233369053.pdf), generated with kicad-footprint-generator")
     (tags diode)
@@
   )
   (module LED_SMD:LED_0603_1608Metric (layer F.Cu)
-    (at 186.695001 102.335001)
+    (at 147.2 86)
     (descr "LED SMD 0603 (1608 Metric), square (rectangular) end terminal, IPC_7351 nominal, (Body size source: http://www.tortai-tech.com/upload/download/2011102023233369053.pdf), generated with kicad-footprint-generator")
     (tags diode)
@@
   )
   (module LED_SMD:LED_0603_1608Metric (layer F.Cu)
-    (at 189.745001 102.335001)
+    (at 147 96)
     (descr "LED SMD 0603 (1608 Metric), square (rectangular) end terminal, IPC_7351 nominal, (Body size source: http://www.tortai-tech.com/upload/download/2011102023233369053.pdf), generated with kicad-footprint-generator")
     (tags diode)
@@
   )
   (module LED_SMD:LED_0603_1608Metric (layer F.Cu)
-    (at 192.795001 102.335001)
+    (at 167 96)
     (descr "LED SMD 0603 (1608 Metric), square (rectangular) end terminal, IPC_7351 nominal, (Body size source: http://www.tortai-tech.com/upload/download/2011102023233369053.pdf), generated with kicad-footprint-generator")
     (tags diode)
@@
   )
   (module LED_SMD:LED_RGB_5050-6 (layer F.Cu)
-    (at 206.625001 83.775001)
+    (at 206.625001 80.6)
     (descr http://cdn.sparkfun.com/datasheets/Components/LED/5060BRG4.pdf)
     (tags "RGB LED 5050-6")
@@
   (gr_arc (start 151 90) (end 151 79) (angle -90) (layer Edge.Cuts) (width 0.15))
   (gr_arc (start 163 90) (end 174 90) (angle -90) (layer Edge.Cuts) (width 0.15))
+  (via (at 156.21 90.297) (size 0.8) (drill 0.4) (layers F.Cu B.Cu) (net 1))
+  (via (at 158.75 96.266) (size 0.8) (drill 0.4) (layers F.Cu B.Cu) (net 1))
 )
