File: Week7Theflower/THEFLOWER.sch (KiCad schematic (older format))
At the start: 6 parts

Commit message: trying to make component choices work
Parts:
- added C1: 1uF, Capacitor_SMD:C_0603_1608Metric, symbol Device:C
- added C2: 100nF, Capacitor_SMD:C_0603_1608Metric, symbol Device:C
- added D10, D7, D8, D9: LED_RGB, LED_SMD:LED_RGB_5050-6, symbol Device:LED_RGB
- added D5, D6: LED, LED_SMD:LED_0603_1608Metric, symbol Device:LED
- added R1: 3k3, Resistor_SMD:R_0603_1608Metric, symbol Device:R
- added U2: SN3218, Package_DFN_QFN:QFN-24_4x4mm_P0.5mm, symbol BAWKiCADLib:SN3218
- BT1: renamed from BT?; footprint (none) -> Battery:BatteryHolder_MPD_BC2003_1x2032
- D1, D2, D3, D4: renamed from D?; footprint (none) -> LED_SMD:LED_0603_1608Metric
- gave numbers to parts that had none: 1
Connections:
- net labels added: +3V3, BACKLED1, BACKLED2, C1B, C1G, C1R, C2B, C2G, C2R, C3B, C3G, C3R, C4B, C4G, C4R, GND, LEAF1, LEAF2, LEAF3, LEAF4
- wire segments 0 -> 87

Commit message: flower updates
Parts:
- added C?: 100nF, Capacitor_SMD:C_0603_1608Metric, symbol Device:C
- added C?: 10nF, Capacitor_SMD:C_0603_1608Metric, symbol Device:C
Connections:
- wire segments 87 -> 96
Changed lines of the file:
@@
 Text Label 6450 2600 0    50   ~ 0
 C4G
+Wire Wire Line
+	4100 3900 4100 4100
+Connection ~ 4100 4100
+Wire Wire Line
+	4100 4100 4100 4600
+$Comp
+L Device:C C?
+U 1 1 5BA75EB3
+P 4550 4350
+F 0 "C?" H 4665 4396 50  0000 L CNN
+F 1 "100nF" H 4665 4305 50  0000 L CNN
+F 2 "Capacitor_SMD:C_0603_1608Metric" H 4588 4200 50  0001 C CNN
+F 3 "~" H 4550 4350 50  0001 C CNN
+	1    4550 4350
+	1    0    0    -1
+$EndComp
+$Comp
+L Device:C C?
+U 1 1 5BA75F65
+P 4950 4350
+F 0 "C?" H 5065 4396 50  0000 L CNN
+F 1 "10nF" H 5065 4305 50  0000 L CNN
+F 2 "Capacitor_SMD:C_0603_1608Metric" H 4988 4200 50  0001 C CNN
+F 3 "~" H 4950 4350 50  0001 C CNN
+	1    4950 4350
+	1    0    0    -1
+$EndComp
+Wire Wire Line
+	4950 4100 4950 4200
+Wire Wire Line
+	4100 4100 4550 4100
+Wire Wire Line
+	4550 4100 4550 4200
+Connection ~ 4550 4100
+Wire Wire Line
+	4550 4100 4950 4100
+Wire Wire Line
+	4550 4500 4550 4550
+Wire Wire Line
+	4950 4500 4950 4550
+$Comp
+L power:GND #PWR?
+U 1 1 5BA81418
+P 4550 4550
+F 0 "#PWR?" H 4550 4300 50  0001 C CNN
+F 1 "GND" H 4555 4377 50  0000 C CNN
+F 2 "" H 4550 4550 50  0001 C CNN
+F 3 "" H 4550 4550 50  0001 C CNN
+	1    4550 4550
+	1    0    0    -1
+$EndComp
+$Comp
+L power:GND #PWR?
+U 1 1 5BA81447
+P 4950 4550
+F 0 "#PWR?" H 4950 4300 50  0001 C CNN
+F 1 "GND" H 4955 4377 50  0000 C CNN
+F 2 "" H 4950 4550 50  0001 C CNN
+F 3 "" H 4950 4550 50  0001 C CNN
+	1    4950 4550
+	1    0    0    -1
+$EndComp
+$Comp
+L power:+3V3 #PWR?
+U 1 1 5BA8155C
+P 4100 3900
+F 0 "#PWR?" H 4100 3750 50  0001 C CNN
+F 1 "+3V3" H 4115 4073 50  0000 C CNN
+F 2 "" H 4100 3900 50  0001 C CNN
+F 3 "" H 4100 3900 50  0001 C CNN
+	1    4100 3900
+	1    0    0    -1
+$EndComp
+$Comp
+L power:GND #PWR?
+U 1 1 5BA817DD
+P 4100 6350
+F 0 "#PWR?" H 4100 6100 50  0001 C CNN
+F 1 "GND" H 4105 6177 50  0000 C CNN
+F 2 "" H 4100 6350 50  0001 C CNN
+F 3 "" H 4100 6350 50  0001 C CNN
+	1    4100 6350
+	1    0    0    -1
+$EndComp
+Wire Wire Line
+	4100 6000 4100 6350
 $EndSCHEMATC
