File: Week-GiveMePower/GiveMePower.kicad_pcb (KiCad board)
At the start: 2 copper layers, 52.5 x 43.5 mm, 21 parts, among them J1 Conn_01x02_Male, J10 Screw_Terminal_01x02, J11 Conn_01x01_Female, J12 Conn_01x01_Female, J13 Conn_01x01_Female, J2 Conn_01x02_Male, J3 Conn_01x02_Male, J4 Conn_01x02_Male, J5 Conn_01x02_Female, J6 Conn_01x02_Female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

Commit message: give me power update
Parts:
- added C1: C, Capacitors_SMD:C_0603, F.Cu at (145.0, 122.2)
- added C4: C, Capacitors_SMD:C_0603, F.Cu at (145.0, 125.5)
- added U1: AP1117-33, TO_SOT_Packages_SMD:SOT-223-3_TabPin2, F.Cu at (139.0, 124.0)
- moved J3 53.2 mm to (105.5, 120.0)
- moved J4 23.6 mm to (110.0, 120.1)
- moved C2 23.1 mm to (113.5, 121.5), turned to 270 degrees
- moved L2 20.2 mm to (117.5, 121.0), turned to 180 degrees
- moved C3 18.6 mm to (121.5, 121.5), turned to 270 degrees
- moved J2 13.7 mm to (125.0, 122.5), turned to 180 degrees
- moved TP3 12.6 mm to (144.0, 135.0)
- moved TP1 12.5 mm to (113.5, 134.5)
- moved TP2 12.5 mm to (136.0, 135.0)
- moved J10 11.0 mm to (127.0, 132.0)
- moved J5 11.0 mm to (105.5, 126.5)
- moved J6 11.0 mm to (149.2, 126.6)
- moved J7 11.0 mm to (127.5, 126.6)
- moved J8 11.0 mm to (105.0, 132.0)
- moved J9 11.0 mm to (149.0, 132.0)
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Connections:
- J10 pad 1: Net-(J10-Pad1) -> /AUXIn
- J10 pad 2: Net-(J10-Pad2) -> /AUXout
- J7 pad 1: Net-(J7-Pad1) -> /AUXIn
- J7 pad 2: Net-(J7-Pad2) -> /AUXout
Other:
- board size 52.5 x 43.5 mm -> 52.5 x 54.5 mm
