File: Week-GiveMePower/GiveMePower.sch (KiCad schematic (older format))
At the start: 23 parts

Commit message: more work on week 7
Parts:
- removed C?: C, symbol Device:C
- removed L?: L, symbol Device:L
- C2, C3: renamed from C?; footprint (none) -> Capacitors_SMD:C_1210
- D1: renamed from D?; footprint (none) -> LEDs:LED_0603
- J1, J2, J3, J4, J5, J6, J7: renamed from J?; footprint (none) -> Pin_Headers:Pin_Header_Straight_1x02_Pitch2.54mm
- J10, J8, J9: renamed from J?; footprint (none) -> TerminalBlocks_Phoenix:TerminalBlock_Phoenix_PT-3.5mm_2pol
- J11, J12, J13: renamed from J?; footprint (none) -> Mounting_Holes:MountingHole_6mm_Pad_Via
- L2: renamed from L?; footprint (none) -> Inductors_SMD:L_Taiyo-Yuden_MD-3030
- R1: renamed from R?; footprint (none) -> Resistors_SMD:R_0603
- TP1, TP2, TP3: renamed from TP?; footprint (none) -> Measurement_Points:Measurement_Point_Square-SMD-Pad_Big

Commit message: give me power update
Parts:
- added C1: C, Capacitors_SMD:C_1210, symbol Device:C
- added C4: C, Capacitors_SMD:C_0603, symbol Device:C
- added TP?: TestPoint_Probe, Measurement_Points:Measurement_Point_Square-SMD-Pad_Big, symbol Connector:TestPoint_Probe
- added U1: AP1117-33, TO_SOT_Packages_SMD:SOT-223-3_TabPin2, symbol Regulator_Linear:AP1117-33
- C3: footprint Capacitors_SMD:C_1210 -> Capacitors_SMD:C_0603
Connections:
- net labels added: AUXIn, AUXout
- wire segments 47 -> 58
Changed lines of the file:
@@
 F 0 "C3" H 6365 1846 50  0000 L CNN
 F 1 "C" H 6365 1755 50  0000 L CNN
-F 2 "Capacitors_SMD:C_1210" H 6288 1650 50  0001 C CNN
+F 2 "Capacitors_SMD:C_0603" H 6288 1650 50  0001 C CNN
 F 3 "~" H 6250 1800 50  0001 C CNN
 	1    6250 1800
@@
 Wire Wire Line
 	3300 7300 3700 7300
+$Comp
+L Regulator_Linear:AP1117-33 U1
+U 1 1 5BAD0627
+P 2750 2050
+F 0 "U1" H 2750 2292 50  0000 C CNN
+F 1 "AP1117-33" H 2750 2201 50  0000 C CNN
+F 2 "TO_SOT_Packages_SMD:SOT-223-3_TabPin2" H 2750 2250 50  0001 C CNN
+F 3 "http://www.diodes.com/datasheets/AP1117.pdf" H 2850 1800 50  0001 C CNN
+	1    2750 2050
+	1    0    0    -1
+$EndComp
+Wire Wire Line
+	2750 2350 2750 2800
+Wire Wire Line
+	3050 2050 3400 2050
+Wire Wire Line
+	2450 2050 2100 2050
+Wire Wire Line
+	1700 2050 1700 1700
+Wire Wire Line
+	2100 2050 2100 2300
+Connection ~ 2100 2050
+Wire Wire Line
+	2100 2050 1700 2050
+Wire Wire Line
+	3400 2050 3400 2300
+Connection ~ 3400 2050
+$Comp
+L Device:C C1
+U 1 1 5BAD4AC3
+P 2100 2450
+F 0 "C1" H 2215 2496 50  0000 L CNN
+F 1 "C" H 2215 2405 50  0000 L CNN
+F 2 "Capacitors_SMD:C_1210" H 2138 2300 50  0001 C CNN
+F 3 "~" H 2100 2450 50  0001 C CNN
+	1    2100 2450
+	1    0    0    -1
+$EndComp
+$Comp
+L Device:C C4
+U 1 1 5BAD4B4D
+P 3400 2450
+F 0 "C4" H 3515 2496 50  0000 L CNN
+F 1 "C" H 3515 2405 50  0000 L CNN
+F 2 "Capacitors_SMD:C_0603" H 3438 2300 50  0001 C CNN
+F 3 "~" H 3400 2450 50  0001 C CNN
+	1    3400 2450
+	1    0    0    -1
+$EndComp
+Wire Wire Line
+	3400 2600 3400 2800
+$Comp
+L power:GND #PWR018
+U 1 1 5BAD8DB7
+P 3400 2800
+F 0 "#PWR018" H 3400 2550 50  0001 C CNN
+F 1 "GND" H 3405 2627 50  0000 C CNN
+F 2 "" H 3400 2800 50  0001 C CNN
+F 3 "" H 3400 2800 50  0001 C CNN
+	1    3400 2800
+	1    0    0    -1
+$EndComp
+$Comp
+L power:GND #PWR017
+U 1 1 5BAD8DF2
+P 2750 2800
+F 0 "#PWR017" H 2750 2550 50  0001 C CNN
+F 1 "GND" H 2755 2627 50  0000 C CNN
+F 2 "" H 2750 2800 50  0001 C CNN
+F 3 "" H 2750 2800 50  0001 C CNN
+	1    2750 2800
+	1    0    0    -1
+$EndComp
+$Comp
+L power:GND #PWR016
+U 1 1 5BAD8E2D
+P 2100 2800
+F 0 "#PWR016" H 2100 2550 50  0001 C CNN
+F 1 "GND" H 2105 2627 50  0000 C CNN
+F 2 "" H 2100 2800 50  0001 C CNN
+F 3 "" H 2100 2800 50  0001 C CNN
+	1    2100 2800
+	1    0    0    -1
+$EndComp
+Wire Wire Line
+	2100 2600 2100 2800
+Wire Wire Line
+	3400 2050 4000 2050
+$Comp
+L power:VCC #PWR015
+U 1 1 5BADB0D8
+P 1700 1700
+F 0 "#PWR015" H 1700 1550 50  0001 C CNN
+F 1 "VCC" H 1717 1873 50  0000 C CNN
+F 2 "" H 1700 1700 50  0001 C CNN
+F 3 "" H 1700 1700 50  0001 C CNN
+	1    1700 1700
+	1    0    0    -1
+$EndComp
+Text Label 4000 2050 2    50   ~ 0
+Output3V3
+Text Label 4750 7200 0    50   ~ 0
+AUXIn
+Text Label 3300 7200 0    50   ~ 0
+AUXIn
+Text Label 3300 7300 0    50   ~ 0
+AUXout
+Text Label 4750 7300 0    50   ~ 0
+AUXout
+$Comp
+L Connector:TestPoint_Probe TP?
+U 1 1 5BADBA21
+P 6050 4250
+F 0 "TP?" H 6203 4352 50  0000 L CNN
+F 1 "TestPoint_Probe" H 6203 4261 50  0000 L CNN
+F 2 "Measurement_Points:Measurement_Point_Square-SMD-Pad_Big" H 6250 4250 50  0001 C CNN
+F 3 "~" H 6250 4250 50  0001 C CNN
+	1    6050 4250
+	1    0    0    -1
+$EndComp
+Wire Wire Line
+	6050 4250 5600 4250
 $EndSCHEMATC
