File: Week-LoraThing/LoraThing.kicad_pcb (KiCad board)
At the start: 2 copper layers, 27 x 43 mm, 33 parts, among them J1 Conn_01x07_Male, J2 Conn_01x07_Male, J3 Conn_01x01_Female, U1 AP7333-33SRG-7, U2 RFM95W-868S2

Commit message: syncing work from lora thing
Routing:
- net /SPI_MISO: track 3.50 -> 36.7 mm
- net /SPI_MOSI: track 3.00 -> 4.19 mm
- net /SPI_SCK: track 3.00 -> 4.09 mm
- net /SPI_CS: track 3.00 -> 4.09 mm
Changed lines of the file:
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@@
     (thickness 1.6)
     (drawings 13)
-    (tracks 185)
+    (tracks 196)
     (zones 0)
     (modules 33)
@@
     (pad_to_mask_clearance 0.2)
     (aux_axis_origin 0 0)
-    (visible_elements FFFFFF7F)
+    (visible_elements 7FFFFFFF)
     (pcbplotparams
       (layerselection 0x010fc_ffffffff)
@@
   (gr_line (start 139 47) (end 137 47) (layer Edge.Cuts) (width 0.2))
   (gr_line (start 139 69) (end 139 49) (layer Edge.Cuts) (width 0.2))
-  (via (at 118.75 62.25) (size 0.8) (drill 0.4) (layers F.Cu B.Cu) (net 38))
-  (via (at 118.75 57.75) (size 0.8) (drill 0.4) (layers F.Cu B.Cu) (net 35))
-  (via (at 120 59.5) (size 0.8) (drill 0.4) (layers F.Cu B.Cu) (net 36))
-  (via (at 120 60.5) (size 0.8) (drill 0.4) (layers F.Cu B.Cu) (net 37))
   (segment (start 120.95 49) (end 121 49) (width 0.25) (layer F.Cu) (net 2))
   (segment (start 120.2 49.75) (end 120.95 49) (width 0.25) (layer F.Cu) (net 2))
@@
   (segment (start 116 64.34) (end 114.3 66.04) (width 0.25) (layer F.Cu) (net 15))
   (segment (start 116 62.8) (end 116 64.34) (width 0.25) (layer F.Cu) (net 15))
-  (via (at 129 61) (size 0.8) (drill 0.4) (layers F.Cu B.Cu) (net 19))
   (segment (start 128.15 65.2) (end 128.15 66.4) (width 0.25) (layer F.Cu) (net 16))
   (segment (start 128.15 66.4) (end 129 67.25) (width 0.25) (layer F.Cu) (net 16))
@@
   (segment (start 128.15 63.6) (end 127.45 63.6) (width 0.25) (layer F.Cu) (net 18))
   (segment (start 127.45 63.6) (end 127.25 63.4) (width 0.25) (layer F.Cu) (net 18))
+  (via (at 129 61) (size 0.8) (drill 0.4) (layers F.Cu B.Cu) (net 19))
   (segment (start 128.15 61.85) (end 129 61) (width 0.25) (layer F.Cu) (net 19))
   (segment (start 128.15 62.8) (end 128.15 61.85) (width 0.25) (layer F.Cu) (net 19))
@@
   (segment (start 121.5 51.50434) (end 124.50434 48.5) (width 0.25) (layer B.Cu) (net 23))
   (segment (start 124.50434 48.5) (end 127 48.5) (width 0.25) (layer B.Cu) (net 23))
-  (via (at 131.25 63.5) (size 0.8) (drill 0.4) (layers F.Cu B.Cu) (net 28))
-  (via (at 131.25 62.5) (size 0.8) (drill 0.4) (layers F.Cu B.Cu) (net 29))
   (via (at 125.75 68) (size 0.8) (drill 0.4) (layers F.Cu B.Cu) (net 24))
   (via (at 125.75 65) (size 0.8) (drill 0.4) (layers F.Cu B.Cu) (net 25))
@@
   (segment (start 124.64075 49) (end 132.75 49) (width 0.25) (layer B.Cu) (net 26))
   (via (at 125.75 62) (size 0.8) (drill 0.4) (layers F.Cu B.Cu) (net 27))
+  (via (at 131.25 63.5) (size 0.8) (drill 0.4) (layers F.Cu B.Cu) (net 28))
   (segment (start 124.35 62) (end 124.35 62.85) (width 0.25) (layer B.Cu) (net 28))
   (segment (start 125 63.5) (end 131.25 63.5) (width 0.25) (layer B.Cu) (net 28))
@@
   (segment (start 133 49.5) (end 135 47.5) (width 0.25) (layer B.Cu) (net 28))
   (segment (start 135 47.5) (end 135 44.75) (width 0.25) (layer B.Cu) (net 28))
+  (via (at 131.25 62.5) (size 0.8) (drill 0.4) (layers F.Cu B.Cu) (net 29))
   (segment (start 124.35 59.85) (end 125 60.5) (width 0.25) (layer B.Cu) (net 29))
   (segment (start 124.35 59) (end 124.35 59.85) (width 0.25) (layer B.Cu) (net 29))
@@
   (segment (start 123 45) (end 123 42.75) (width 0.25) (layer F.Cu) (net 29))
   (segment (start 123 42.75) (end 123 42.75) (width 0.25) (layer F.Cu) (net 29))
-  (via (at 123 42.75) (size 0.8) (drill 0.4) (layers F.Cu B.Cu) (net 29))
   (segment (start 124.35 59) (end 123 57.65) (width 0.25) (layer B.Cu) (net 29))
-  (segment (start 123 51.91357) (end 124.91357 50) (width 0.25) (layer B.Cu) (net 29))
-  (segment (start 123 52.5) (end 123 51.91357) (width 0.25) (layer B.Cu) (net 29))
   (segment (start 123 52.5) (end 123 52.25) (width 0.25) (layer B.Cu) (net 29))
   (segment (start 123 57.65) (end 123 52.5) (width 0.25) (layer B.Cu) (net 29))
-  (segment (start 124.91357 50) (end 133.25 50) (width 0.25) (layer B.Cu) (net 29))
-  (segment (start 133.25 50) (end 135.5 47.75) (width 0.25) (layer B.Cu) (net 29))
-  (segment (start 135.5 47.75) (end 135.5 41.5) (width 0.25) (layer B.Cu) (net 29))
-  (segment (start 133.5 39.5) (end 126.88641 39.5) (width 0.25) (layer B.Cu) (net 29))
-  (segment (start 135.5 41.5) (end 133.5 39.5) (width 0.25) (layer B.Cu) (net 29))
-  (segment (start 126.88641 39.5) (end 126 40.38641) (width 0.25) (layer B.Cu) (net 29))
-  (segment (start 126 40.38641) (end 126 46.5) (width 0.25) (layer B.Cu) (net 29))
-  (segment (start 126 46.5) (end 125.75 46.75) (width 0.25) (layer B.Cu) (net 29))
-  (segment (start 125.75 46.75) (end 124 46.75) (width 0.25) (layer B.Cu) (net 29))
-  (segment (start 123 45.75) (end 123 42.75) (width 0.25) (layer B.Cu) (net 29))
-  (segment (start 124 46.75) (end 123 45.75) (width 0.25) (layer B.Cu) (net 29))
+  (segment (start 124 46.75) (end 123 45.75) (width 0.25) (layer B.Cu) (net 29) (status 1000000))
+  (segment (start 123 45.75) (end 123 42.75) (width 0.25) (layer B.Cu) (net 29) (status 1000000))
+  (segment (start 125.75 46.75) (end 124 46.75) (width 0.25) (layer B.Cu) (net 29) (status 1000000))
+  (segment (start 126 46.5) (end 125.75 46.75) (width 0.25) (layer B.Cu) (net 29) (status 1000000))
+  (segment (start 126 40.38641) (end 126 46.5) (width 0.25) (layer B.Cu) (net 29) (status 1000000))
+  (segment (start 126.88641 39.5) (end 126 40.38641) (width 0.25) (layer B.Cu) (net 29) (status 1000000))
+  (segment (start 135.5 41.5) (end 133.5 39.5) (width 0.25) (layer B.Cu) (net 29) (status 1000000))
+  (segment (start 133.5 39.5) (end 126.88641 39.5) (width 0.25) (layer B.Cu) (net 29) (status 1000000))
+  (segment (start 135.5 47.75) (end 135.5 41.5) (width 0.25) (layer B.Cu) (net 29) (status 1000000))
+  (segment (start 133.25 50) (end 135.5 47.75) (width 0.25) (layer B.Cu) (net 29) (status 1000000))
+  (segment (start 124.91357 50) (end 133.25 50) (width 0.25) (layer B.Cu) (net 29) (status 1000000))
+  (segment (start 123 52.5) (end 123 51.91357) (width 0.25) (layer B.Cu) (net 29) (status 1000000))
+  (segment (start 123 51.91357) (end 124.91357 50) (width 0.25) (layer B.Cu) (net 29) (status 1000000))
+  (via (at 123 42.75) (size 0.8) (drill 0.4) (layers F.Cu B.Cu) (net 29) (status 1000000))
   (via (at 125.75 59) (size 0.8) (drill 0.4) (layers F.Cu B.Cu) (net 30))
-  (via (at 125.75 53) (size 0.8) (drill 0.4) (layers F.Cu B.Cu) (net 34))
   (via (at 125.75 56) (size 0.8) (drill 0.4) (layers F.Cu B.Cu) (net 31))
   (segment (start 125 45) (end 125 43.75) (width 0.25) (layer F.Cu) (net 32))
@@
   (segment (start 121 30.75) (end 121 30.75) (width 0.25) (layer F.Cu) (net 33))
   (via (at 121 30.75) (size 0.8) (drill 0.4) (layers F.Cu B.Cu) (net 33))
+  (via (at 125.75 53) (size 0.8) (drill 0.4) (layers F.Cu B.Cu) (net 34))
+  (via (at 118.75 57.75) (size 0.8) (drill 0.4) (layers F.Cu B.Cu) (net 35))
   (segment (start 125 29) (end 125 32) (width 0.25) (layer F.Cu) (net 35))
   (segment (start 125 32) (end 125 32) (width 0.25) (layer F.Cu) (net 35))
   (via (at 125 32) (size 0.8) (drill 0.4) (layers F.Cu B.Cu) (net 35))
+  (segment (start 118.85 57.85) (end 118.75 57.75) (width 0.25) (layer F.Cu) (net 35))
+  (segment (start 118.85 58.8) (end 118.85 57.85) (width 0.25) (layer F.Cu) (net 35))
+  (via (at 120 59.5) (size 0.8) (drill 0.4) (layers F.Cu B.Cu) (net 36))
   (segment (start 131 29) (end 131 32) (width 0.25) (layer F.Cu) (net 36))
   (segment (start 131 31.75) (end 131 32) (width 0.25) (layer F.Cu) (net 36))
   (segment (start 131 32) (end 131 31.75) (width 0.25) (layer F.Cu) (net 36))
   (via (at 131 32) (size 0.8) (drill 0.4) (layers F.Cu B.Cu) (net 36))
+  (segment (start 119.9 59.6) (end 120 59.5) (width 0.25) (layer F.Cu) (net 36))
+  (segment (start 118.85 59.6) (end 119.9 59.6) (width 0.25) (layer F.Cu) (net 36))
+  (segment (start 120 59.5) (end 121.04999 58.45001) (width 0.25) (layer B.Cu) (net 36))
+  (segment (start 121.04999 41.95001) (end 131 32) (width 0.25) (layer B.Cu) (net 36))
+  (segment (start 121.04999 58.45001) (end 121.04999 41.95001) (width 0.25) (layer B.Cu) (net 36))
+  (via (at 120 60.5) (size 0.8) (drill 0.4) (layers F.Cu B.Cu) (net 37))
   (segment (start 129 29) (end 129 32) (width 0.25) (layer F.Cu) (net 37))
   (segment (start 129 32) (end 129 32) (width 0.25) (layer F.Cu) (net 37))
   (via (at 129 32) (size 0.8) (drill 0.4) (layers F.Cu B.Cu) (net 37))
+  (segment (start 119.9 60.4) (end 120 60.5) (width 0.25) (layer F.Cu) (net 37))
+  (segment (start 118.85 60.4) (end 119.9 60.4) (width 0.25) (layer F.Cu) (net 37))
+  (via (at 118.75 62.25) (size 0.8) (drill 0.4) (layers F.Cu B.Cu) (net 38))
   (segment (start 127 29) (end 127 32) (width 0.25) (layer F.Cu) (net 38))
   (segment (start 127 32) (end 127 32) (width 0.25) (layer F.Cu) (net 38))
   (via (at 127 32) (size 0.8) (drill 0.4) (layers F.Cu B.Cu) (net 38))
+  (segment (start 118.85 62.15) (end 118.75 62.25) (width 0.25) (layer F.Cu) (net 38))
+  (segment (start 118.85 61.2) (end 118.85 62.15) (width 0.25) (layer F.Cu) (net 38))
 )

Commit message: Resyn forgot to save first (again)
Parts:
- moved J2 3.59 mm to (133.6, 68.6)
- moved J1 1.00 mm to (113.3, 68.6)
- renumbered JP3 to eJP3
Routing:
- net /SPI_SCK: track 4.09 -> 37.8 mm
- net /SPI_MOSI: track 4.19 -> 37.4 mm
- net /RESET: track 3.00 -> 32.2 mm, vias 1 -> 2
- net /SPI_CS: track 4.09 -> 32.4 mm
- net VCC: track 2.31 -> 23.7 mm, vias 0 -> 1
- net /GPIO4: track 64.3 -> 48.8 mm
- net /EXT_GPIO6: track 0.00 -> 10.5 mm
- net +3V3: track 11.3 -> 20.1 mm
- net /EXT_GPIO5: track 0.00 -> 6.59 mm
- net /GPIO2: track 47.4 -> 41.2 mm
- net /GPIO3: track 42.5 -> 37.5 mm
- net /GPIO6: track 48.5 -> 52.6 mm, vias 1 -> 2
- net /ANTENNA: track 0.00 -> 4.00 mm
- net /EXT_GPIO2: track 14.8 -> 11.0 mm
- net /EXT_GPIO4: track 10.6 -> 7.27 mm
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- added copper zone on B.Cu, net GND
- added copper zone on F.Cu, net GND
Other:
- board size 27 x 43 mm -> 24 x 43 mm

Commit message: lora thing complete
Parts:
- added G***: LOGO, ArtworkAndSilks:frontside, F.Cu at (124.0, 50.0)
- added G***: LOGO, ArtworkAndSilks:backside, B.Cu at (123.3, 49.4)
Routing:
- net /SPI_EXT_SCK: track 6.02 -> 7.02 mm
- net /SPI_EXT_MOSI: track 4.54 -> 5.54 mm
- net /SPI_EXT_MISO: track 3.41 -> 4.41 mm
- net /RESET: track 32.2 -> 33.2 mm
- net /SPI_EXT_CS: track 3.01 -> 4.01 mm
- net VCC: track 23.7 -> 24.7 mm
