File: Week-M0GO/_saved_mogo.sch (KiCad schematic (older format))
At the start: 8 parts

Commit message: finish schmatic m0go
Parts:
- added BT1: Battery_Cell, symbol Device:Battery_Cell
- added C1, C10, C2, C3, C4, C5, C6, C7, C8, C9: C, symbol Device:C
- added D1, D2: DIODE, symbol pspice:DIODE
- added J2: Conn_01x06_Female, symbol Connector:Conn_01x06_Female
- added J3, J4: Conn_01x20_Female, symbol Connector:Conn_01x20_Female
- added Q1: Q_PMOS_GDS, symbol Device:Q_PMOS_GDS
- added R1, R2, R5, R6, R8: R, symbol Device:R
- added Y2: Crystal 32.76 Khz, symbol Device:Crystal
- Y1: renamed from Y?; value Crystal -> Crystal 8Mhz
- gave numbers to parts that had none: 7
Connections:
- net labels added: +BATT, OSC_IN, OSC_OUT, PB0, PB1, PB10, PB11, PB12, PB13, PB14, PB15, PB2, PB3, PB5, PB6, PB7, PB8, PB9, PC13, RTC_OSC_IN, RTC_OSC_OUT
- net labels removed: +5V
- wire segments 62 -> 186
Other:
- moved on the sheet: U1
