File: Week-M0GO/mogo.sch (KiCad schematic (older format))
At the start: 4 parts

Commit message: More schematic work
Parts:
- removed U?: 25LCxxx, symbol Memory_EEPROM:25LCxxx
- added R? (x3): R, symbol Device:R
- added U?: CAT24C256, symbol Memory_EEPROM:CAT24C256
Connections:
- net labels added: BOOT0, OTG_SELECT, SCL_3V3, SDA_3V3, USB_D+, USB_D-, _RESET
- wire segments 0 -> 58

Commit message: Added Lora Thing schmatic and almost finished board
Parts:
- added U?: AP7333-33SRG-7, TO_SOT_Packages_SMD:SOT-23, symbol BAWKiCADLib:AP7333-33SRG-7
Changed lines of the file:
@@
 Text Label 3850 4100 2    50   ~ 0
 SCL_3V3
+$Comp
+L BAWKiCADLib:AP7333-33SRG-7 U?
+U 1 1 5BC0C074
+P 9350 3050
+F 0 "U?" H 9350 3342 50  0000 C CNN
+F 1 "AP7333-33SRG-7" H 9350 3251 50  0000 C CNN
+F 2 "TO_SOT_Packages_SMD:SOT-23" H 9400 3400 50  0001 C CNN
+F 3 "https://www.diodes.com/assets/Datasheets/AP7333.pdf" H 9600 3500 50  0001 C CNN
+	1    9350 3050
+	1    0    0    -1
+$EndComp
 $EndSCHEMATC

Commit message: m0go SCHEMATIC WORK
Connections:
- net labels added: PA0, PA1, PA10, PA15, PA2, PA3, PA4, PA5, PA6, PA7, PA8, PA9, SWCLK, SWDIO
- wire segments 58 -> 62

Commit message: finish schmatic m0go
Parts:
- added BT?: Battery_Cell, symbol Device:Battery_Cell
- added C? (x10): C, symbol Device:C
- added D? (x2): DIODE, symbol pspice:DIODE
- added Q?: Q_PMOS_GDS, symbol Device:Q_PMOS_GDS
- added R? (x5): R, symbol Device:R
- added Y?: Crystal 32.76 Khz, symbol Device:Crystal
- Y?: value Crystal -> Crystal 8Mhz
Connections:
- net labels added: +BATT, OSC_IN, OSC_OUT, PB0, PB1, PB10, PB11, PB12, PB13, PB14, PB15, PB2, PB3, PB5, PB6, PB7, PB8, PB9, RTC_OSC_IN, RTC_OSC_OUT
- net labels removed: +5V
- wire segments 62 -> 135
Other:
- moved on the sheet: U?

Commit message: resync
Parts:
- added J2: Conn_01x06_Female, Pin_Headers:Pin_Header_Straight_1x05_Pitch2.54mm, symbol Connector:Conn_01x06_Female
- added J3, J4: Conn_01x20_Female, Pin_Headers:Pin_Header_Straight_1x20_Pitch2.54mm, symbol Connector:Conn_01x20_Female
- BT1: renamed from BT?; footprint (none) -> Battery_Holders:Keystone_1058_1x2032-CoinCell
- C1, C10, C2, C3, C4, C5, C6, C7, C8, C9: renamed from C?; footprint (none) -> Capacitors_SMD:C_0603
- D1, D2: renamed from D?; footprint (none) -> Diodes_SMD:D_SOD-323F
- J1: renamed from J?; footprint (none) -> Connectors_USB:USB_Micro-B_Molex-105017-0001
- Q1: renamed from Q?; footprint (none) -> TO_SOT_Packages_SMD:SOT-23
- R1, R2, R3, R4, R5, R6, R7, R8: renamed from R?; footprint (none) -> Resistors_SMD:R_0603
- U1: renamed from U?; footprint (none) -> Housings_SOIC:SOIC-8_3.9x4.9mm_Pitch1.27mm
- U2: renamed from U?; footprint Package_QFP:LQFP-48_7x7mm_P0.5mm -> Housings_QFP:LQFP-48_7x7mm_Pitch0.5mm
- Y1: renamed from Y?; footprint (none) -> Crystals:Crystal_SMD_3225-4pin_3.2x2.5mm
- Y2: renamed from Y?; footprint (none) -> Crystals:Crystal_Round_d1.0mm_Vertical
- gave numbers to parts that had none: 1
Connections:
- net labels added: PC13
- wire segments 135 -> 186

Commit message: started routing
Parts:
- added SW1: SW_Push, Button_Switch_SMD:SW_SPST_TL3342, symbol Switch:SW_Push
- J2: footprint Pin_Headers:Pin_Header_Straight_1x05_Pitch2.54mm -> Connector_PinHeader_2.54mm:PinHeader_1x06_P2.54mm_Vertical
Connections:
- net labels added: PB4
- wire segments 186 -> 189
Changed lines of the file:
@@
 PB3
 Text Label 5250 3500 0    50   ~ 0
-PB3
+PB4
 Text Label 5250 3600 0    50   ~ 0
 PB5
@@
 F 0 "J2" H 4277 4676 50  0000 L CNN
 F 1 "Conn_01x06_Female" H 4277 4585 50  0000 L CNN
-F 2 "Pin_Headers:Pin_Header_Straight_1x05_Pitch2.54mm" H 4250 4700 50  0001 C CNN
+F 2 "Connector_PinHeader_2.54mm:PinHeader_1x06_P2.54mm_Vertical" H 4250 4700 50  0001 C CNN
 F 3 "~" H 4250 4700 50  0001 C CNN
 	1    4250 4700
@@
 PB3
 Text Label 4050 6550 0    50   ~ 0
-PB3
+PB4
 Text Label 4050 6650 0    50   ~ 0
 PB5
@@
 	1    0    0    -1
 $EndComp
+$Comp
+L Switch:SW_Push SW1
+U 1 1 5BE7EB70
+P 3500 2250
+F 0 "SW1" H 3500 2535 50  0000 C CNN
+F 1 "SW_Push" H 3500 2444 50  0000 C CNN
+F 2 "Button_Switch_SMD:SW_SPST_TL3342" H 3500 2450 50  0001 C CNN
+F 3 "" H 3500 2450 50  0001 C CNN
+	1    3500 2250
+	1    0    0    -1
+$EndComp
+Wire Wire Line
+	3700 2250 4150 2250
+Wire Wire Line
+	3300 2250 3050 2250
+Wire Wire Line
+	3050 2250 3050 2500
+Text Label 4150 2250 2    50   ~ 0
+_RESET
+$Comp
+L power:GND #PWR0103
+U 1 1 5BE93BB2
+P 3050 2500
+F 0 "#PWR0103" H 3050 2250 50  0001 C CNN
+F 1 "GND" H 3055 2327 50  0000 C CNN
+F 2 "" H 3050 2500 50  0001 C CNN
+F 3 "" H 3050 2500 50  0001 C CNN
+	1    3050 2500
+	1    0    0    -1
+$EndComp

Commit message: board work m0go
Parts:
- removed Y1: Crystal 8Mhz, Crystals:Crystal_SMD_3225-4pin_3.2x2.5mm, symbol Device:Crystal
- added Y1: Crystal_GND24, symbol Device:Crystal_GND24
Changed lines of the file:
@@
 $EndComp
 $Comp
-L Device:Crystal Y1
-U 1 1 5BBCD0D5
-P 1300 6800
-F 0 "Y1" H 1300 7068 50  0000 C CNN
-F 1 "Crystal 8Mhz" H 1300 6977 50  0000 C CNN
-F 2 "Crystals:Crystal_SMD_3225-4pin_3.2x2.5mm" H 1300 6800 50  0001 C CNN
-F 3 "~" H 1300 6800 50  0001 C CNN
-	1    1300 6800
-	1    0    0    -1
-$EndComp
-$Comp
 L power:GND #PWR0101
 U 1 1 5BBCD1D2
@@
 	6200 7400 5800 7400
 Wire Wire Line
+	4450 7450 4050 7450
+Wire Wire Line
+	4450 7550 4050 7550
+Wire Wire Line
 	4450 5750 4050 5750
 Wire Wire Line
@@
 	4450 5950 4050 5950
 Wire Wire Line
+	4450 6050 4050 6050
+Wire Wire Line
 	4450 6150 4050 6150
 Wire Wire Line
@@
 	4450 7250 4050 7250
 Wire Wire Line
-	4450 7350 4050 7350
-Wire Wire Line
-	4450 7450 4050 7450
-Wire Wire Line
-	4450 7550 4050 7550
-Wire Wire Line
-	4450 7650 4050 7650
-Wire Wire Line
 	5800 7500 6200 7500
 Wire Wire Line
@@
 Text Label 3650 4900 0    50   ~ 0
 BOOT0
-Text Label 4050 6150 0    50   ~ 0
+Text Label 5800 6900 0    50   ~ 0
 PB0
-Text Label 4050 6250 0    50   ~ 0
+Text Label 5800 7000 0    50   ~ 0
 PB1
-Text Label 4050 6350 0    50   ~ 0
+Text Label 5800 7100 0    50   ~ 0
 PB2
-Text Label 4050 6450 0    50   ~ 0
+Text Label 4050 6650 0    50   ~ 0
 PB3
-Text Label 4050 6550 0    50   ~ 0
+Text Label 4050 6750 0    50   ~ 0
 PB4
-Text Label 4050 6650 0    50   ~ 0
+Text Label 4050 6850 0    50   ~ 0
 PB5
-Text Label 4050 6750 0    50   ~ 0
+Text Label 4050 6950 0    50   ~ 0
 PB6
-Text Label 4050 6850 0    50   ~ 0
+Text Label 4050 7050 0    50   ~ 0
 PB7
-Text Label 4050 6950 0    50   ~ 0
+Text Label 4050 7150 0    50   ~ 0
 PB8
-Text Label 4050 7050 0    50   ~ 0
+Text Label 4050 7250 0    50   ~ 0
 PB9
-Text Label 4050 7150 0    50   ~ 0
+Text Label 5800 7200 0    50   ~ 0
 PB10
-Text Label 4050 7250 0    50   ~ 0
+Text Label 5800 7300 0    50   ~ 0
 PB11
-Text Label 4050 7350 0    50   ~ 0
+Text Label 5800 7400 0    50   ~ 0
 PB12
-Text Label 4050 7450 0    50   ~ 0
+Text Label 5800 7500 0    50   ~ 0
 PB13
-Text Label 4050 7550 0    50   ~ 0
+Text Label 5800 7600 0    50   ~ 0
 PB14
-Text Label 4050 7650 0    50   ~ 0
+Text Label 4050 5750 0    50   ~ 0
 PB15
 Text Label 5800 6200 0    50   ~ 0
@@
 Text Label 5800 6800 0    50   ~ 0
 PA7
-Text Label 5800 6900 0    50   ~ 0
+Text Label 4050 5850 0    50   ~ 0
 PA8
-Text Label 5800 7000 0    50   ~ 0
+Text Label 4050 5950 0    50   ~ 0
 PA9
-Text Label 5800 7100 0    50   ~ 0
+Text Label 4050 6050 0    50   ~ 0
 PA10
 Wire Wire Line
@@
 	5800 6100 6200 6100
 Wire Wire Line
-	4050 5750 4050 5600
+	3850 7350 3850 7200
 Wire Wire Line
 	5800 5700 5800 5550
@@
 L power:+BATT #PWR013
 U 1 1 5C0046D8
-P 4050 5600
-F 0 "#PWR013" H 4050 5450 50  0001 C CNN
-F 1 "+BATT" H 4065 5773 50  0000 C CNN
-F 2 "" H 4050 5600 50  0001 C CNN
-F 3 "" H 4050 5600 50  0001 C CNN
-	1    4050 5600
+P 3850 7200
+F 0 "#PWR013" H 3850 7050 50  0001 C CNN
+F 1 "+BATT" H 3865 7373 50  0000 C CNN
+F 2 "" H 3850 7200 50  0001 C CNN
+F 3 "" H 3850 7200 50  0001 C CNN
+	1    3850 7200
 	1    0    0    -1
 $EndComp
-Text Label 4050 5850 0    50   ~ 0
+Text Label 4050 7450 0    50   ~ 0
 _RESET
-Text Label 4050 5950 0    50   ~ 0
+Text Label 4050 7550 0    50   ~ 0
 BOOT0
-Text Label 5800 7200 0    50   ~ 0
+Text Label 4050 6150 0    50   ~ 0
 USB_D-
-Text Label 5800 7300 0    50   ~ 0
+Text Label 4050 6250 0    50   ~ 0
 USB_D+
-Text Label 5800 7400 0    50   ~ 0
+Text Label 4050 6350 0    50   ~ 0
 SWDIO
-Text Label 5800 7500 0    50   ~ 0
+Text Label 4050 6450 0    50   ~ 0
 SWCLK
-Text Label 5800 7600 0    50   ~ 0
+Text Label 4050 6550 0    50   ~ 0
 PA15
 Text Label 5150 2800 0    50   ~ 0
@@
 PC13
 Wire Wire Line
-	3700 6050 3700 5800
+	3700 7650 3700 7400
 Wire Wire Line
-	3700 6050 4450 6050
+	3700 7650 4450 7650
 $Comp
 L power:VBUS #PWR012
 U 1 1 5C03831E
-P 3700 5800
-F 0 "#PWR012" H 3700 5650 50  0001 C CNN
-F 1 "VBUS" H 3715 5973 50  0000 C CNN
-F 2 "" H 3700 5800 50  0001 C CNN
-F 3 "" H 3700 5800 50  0001 C CNN
-	1    3700 5800
+P 3700 7400
+F 0 "#PWR012" H 3700 7250 50  0001 C CNN
+F 1 "VBUS" H 3715 7573 50  0000 C CNN
+F 2 "" H 3700 7400 50  0001 C CNN
+F 3 "" H 3700 7400 50  0001 C CNN
+	1    3700 7400
 	1    0    0    -1
 $EndComp
@@
 	1    0    0    -1
 $EndComp
+Wire Wire Line
+	3850 7350 4450 7350
+$Comp
+L Device:Crystal_GND24 Y1
+U 1 1 5C0DB3F5
+P 1300 6800
+F 0 "Y1" H 1491 6846 50  0000 L CNN
+F 1 "Crystal_GND24" H 1491 6755 50  0000 L CNN
+F 2 "" H 1300 6800 50  0001 C CNN
+F 3 "~" H 1300 6800 50  0001 C CNN
+	1    1300 6800
+	1    0    0    -1
+$EndComp
+$Comp
+L power:GND #PWR0107
+U 1 1 5C0DB51C
+P 1300 7000
+F 0 "#PWR0107" H 1300 6750 50  0001 C CNN
+F 1 "GND" H 1305 6827 50  0000 C CNN
+F 2 "" H 1300 7000 50  0001 C CNN
+F 3 "" H 1300 7000 50  0001 C CNN
+	1    1300 7000
+	1    0    0    -1
+$EndComp
+$Comp
+L power:GND #PWR0108
+U 1 1 5C0DB567
+P 1300 6600
+F 0 "#PWR0108" H 1300 6350 50  0001 C CNN
+F 1 "GND" H 1305 6427 50  0000 C CNN
+F 2 "" H 1300 6600 50  0001 C CNN
+F 3 "" H 1300 6600 50  0001 C CNN
+	1    1300 6600
+	-1   0    0    1
+$EndComp
 $EndSCHEMATC

Commit message: mogo routing finished
Changed lines of the file:
@@
 	5650 4200 5250 4200
-Wire Wire Line
-	5650 4300 5250 4300
-Wire Wire Line
-	5650 4400 5250 4400
-Wire Wire Line
-	5650 4500 5250 4500
 Wire Wire Line
 	5650 4600 5250 4600
@@
 	-1   0    0    1
 $EndComp
+Wire Wire Line
+	4800 4400 5650 4400
+Text Label 4800 4400 2    50   ~ 0
+SDA_3V3
+Text Label 4800 4500 2    50   ~ 0
+SCL_3V3
+Wire Wire Line
+	4800 4500 5650 4500
+Wire Wire Line
+	5250 4300 5650 4300
 $EndSCHEMATC
