File: WeekBUBBLEWATCHreborn/BubbleWatch.kicad_pcb (KiCad board)
At the start: 2 copper layers, 84 x 38 mm, 38 parts, among them J1 Conn_02x02_Counter_Clockwise, J2 Conn_02x02_Counter_Clockwise, J3 Conn_01x05, SW1 SW_Push, SW2 SW_Push, SW3 SW_Push, SW4 SW_Push, U1 RedRetroBubbleDisplay, U2 RedRetroBubbleDisplay, U3 STM32F030C8Tx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

Commit message: Bubblewathc reborn routing finished
Parts:
- J3: footprint Connector_Harwin:Harwin_M20-89005xx_1x05_P2.54mm_Horizontal -> Connector_Harwin:Harwin_M20-89010xx_1x10_P2.54mm_Horizontal
- moved SW2 16.6 mm to (158.8, 74.0)
- moved SW4 16.5 mm to (158.8, 89.7)
- moved J3 5.26 mm to (144.0, 66.5)
Connections:
- J3 pad 2: /RESET -> GND
- J3 pad 3: /SWDIO -> /I2C1_SCL
- J3 pad 4: /SWDCLK -> /I2C1_SDA
- SW1 pad 1: Net-(SW1-Pad1) -> GND
- SW2 pad 1: Net-(SW1-Pad1) -> GND
- SW3 pad 1: Net-(SW1-Pad1) -> GND
- SW4 pad 1: Net-(SW1-Pad1) -> GND
- U3 pad 12: /BUTTON1 -> (no net)
- U3 pad 13: /BUTTON2 -> (no net)
- U3 pad 14: /BUTTON3 -> (no net)
- U3 pad 15: /BUTTON4 -> (no net)
- U3 pad 39: Net-(U3-Pad39) -> /BUTTON4
- U3 pad 45: Net-(U3-Pad45) -> /BUTTON3
- U3 pad 46: Net-(U3-Pad46) -> /BUTTON2
Routing:
- net (no net): track 19.9 -> 56.9 mm, vias 1 -> 4
- net +3V3: track 65.6 -> 98.5 mm, vias 2 -> 3
- net /I2C1_SDA: track 3.55 -> 30.4 mm, vias 0 -> 1
- net +BATT: track 25.4 -> 50.0 mm
- net Net-(U3-Pad17): track 0.00 -> 24.1 mm, vias 0 -> 1
- net Net-(U3-Pad16): track 0.00 -> 21.3 mm, vias 0 -> 1
- net /BUTTON1: track 0.00 -> 19.1 mm, vias 0 -> 1
- net /BUTTON4: track 0.00 -> 13.8 mm, vias 0 -> 1
- net /BUTTON2: track 0.00 -> 13.3 mm, vias 0 -> 1
- net /BUTTON3: track 0.00 -> 9.49 mm, vias 0 -> 1
- net /I2C1_SCL: track 25.6 -> 32.4 mm
- net /SEGB: track 43.7 -> 42.7 mm
- net /RESET: track 24.8 -> 25.6 mm
- net GND: vias 0 -> 14
- added copper zone on B.Cu, net GND
