File: WeekBUBBLEWATCHreborn/_autosave-BubbleWatch.kicad_pcb (KiCad board)
At the start: 2 copper layers, 84 x 38 mm, 38 parts, among them J1 Conn_02x02_Counter_Clockwise, J2 Conn_02x02_Counter_Clockwise, J3 Conn_01x05, SW1 SW_Push, SW2 SW_Push, SW3 SW_Push, SW4 SW_Push, U1 RedRetroBubbleDisplay, U2 RedRetroBubbleDisplay, U3 STM32F030C8Tx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

Commit message: Bubblewathc reborn routing finished
Routing:
- net +BATT: track 29.0 -> 50.0 mm
- net GND: vias 11 -> 14
