File: Week-Rain/rain.kicad_pcb (KiCad board)
At the start: 2 copper layers, 49 x 26 mm, 24 parts, among them J1 Conn_01x06_Female, J2 Micro_SD_Card_Det, J3 Conn_01x04_Female, U1 AP7333-28SRG-7, U2 BME680, U3 RFM95W-868S2, U4 STM32L011F4Ux

Commit message: Rain silks and gerber done
Parts:
- added G***: LOGO, ArtAndSilks:topsilk, F.Cu at (119.5, 92.0)
- added G***: LOGO, ArtAndSilks:botsilk, B.Cu at (113.5, 88.0)
