File: Week-HDMY/HDMY.sch (KiCad schematic (older format))
At the start: 4 parts

Commit message: almost completed HDMY schematic
Parts:
- added C1, C2, C3, C4, C5: 1uF, symbol Device:C_Small
- added J?: Conn_01x10, symbol Connector_Generic:Conn_01x10
- added JP1, JP10, JP2, JP3, JP4, JP5, JP6, JP7, JP8, JP9: SolderJumper_2_Bridged, Jumper:SolderJumper-2_P1.3mm_Bridged_RoundedPad1.0x1.5mm, symbol Jumper:SolderJumper_2_Bridged
- added R1, R2: 4K7, symbol Device:R_Small
- added U2: AP7333-33SRG-7, TO_SOT_Packages_SMD:SOT-23, symbol BAWKiCADLib:AP7333-33SRG-7
- added U3: AP7333-15SRG-7, TO_SOT_Packages_SMD:SOT-23, symbol BAWKiCADLib:AP7333-33SRG-7
- gave numbers to parts that had none: 4
Connections:
- net labels added: +1V5, +3V3, INACEC, INAHBD, INASCL, INASDA, INAUTIL, INBCEC, INBCLK+, INBCLK-, INBD0+, INBD0-, INBD1+, INBD1-, INBD2+, INBD2-, INBHBD, INBSCL, INBSDA, INBUTIL, SELECT
- wire segments 81 -> 196
Other:
- note added: "Input Ports \n"

Commit message: completed schmatic working on layout for HDMY
Parts:
- added R3: 1K8, Resistor_SMD:R_0603_1608Metric, symbol Device:R_Small
- added R4: 1K5, Resistor_SMD:R_0603_1608Metric, symbol Device:R_Small
- C1, C2, C3, C4, C5: footprint (none) -> Capacitor_SMD:C_0603_1608Metric
- J1, J2, J3: footprint (none) -> Connector_HDMI:HDMI_A_Contact_Technology_HDMI-19APL2_Horizontal
- J4: renamed from J?; footprint (none) -> Connector_PinHeader_2.54mm:PinHeader_1x10_P2.54mm_Vertical
- R1, R2: footprint (none) -> Resistor_SMD:R_0603_1608Metric
- U1: footprint (none) -> Package_SO:TSSOP-48_6.1x12.5mm_P0.5mm
- U2, U3: footprint TO_SOT_Packages_SMD:SOT-23 -> Package_TO_SOT_SMD:SOT-23
Connections:
- net labels added: OUTSEL
- wire segments 196 -> 216
Changed lines of the file:
@@
 F 0 "U1" H 3550 1000 50  0000 C CNN
 F 1 "TS3DV421" H 3650 3300 50  0000 C CNN
-F 2 "" H 3300 2150 50  0001 C CNN
+F 2 "Package_SO:TSSOP-48_6.1x12.5mm_P0.5mm" H 3300 2150 50  0001 C CNN
 F 3 "" H 3300 2150 50  0001 C CNN
 	1    3300 2150
@@
 F 0 "J1" H 2180 5596 50  0000 L CNN
 F 1 "HDMI_A" H 2180 5505 50  0000 L CNN
-F 2 "" H 1775 5550 50  0001 C CNN
+F 2 "Connector_HDMI:HDMI_A_Contact_Technology_HDMI-19APL2_Horizontal" H 1775 5550 50  0001 C CNN
 F 3 "https://en.wikipedia.org/wiki/HDMI" H 1775 5550 50  0001 C CNN
 	1    1750 5550
@@
 F 0 "J3" H 10630 3346 50  0000 L CNN
 F 1 "HDMI_A" H 10630 3255 50  0000 L CNN
-F 2 "" H 10225 3300 50  0001 C CNN
+F 2 "Connector_HDMI:HDMI_A_Contact_Technology_HDMI-19APL2_Horizontal" H 10225 3300 50  0001 C CNN
 F 3 "https://en.wikipedia.org/wiki/HDMI" H 10225 3300 50  0001 C CNN
 	1    10200 3300
@@
 F 0 "J2" H 8580 3346 50  0000 L CNN
 F 1 "HDMI_A" H 8580 3255 50  0000 L CNN
-F 2 "" H 8175 3300 50  0001 C CNN
+F 2 "Connector_HDMI:HDMI_A_Contact_Technology_HDMI-19APL2_Horizontal" H 8175 3300 50  0001 C CNN
 F 3 "https://en.wikipedia.org/wiki/HDMI" H 8175 3300 50  0001 C CNN
 	1    8150 3300
@@
 F 0 "U2" H 4900 4342 50  0000 C CNN
 F 1 "AP7333-33SRG-7" H 4900 4251 50  0000 C CNN
-F 2 "TO_SOT_Packages_SMD:SOT-23" H 4950 4400 50  0001 C CNN
+F 2 "Package_TO_SOT_SMD:SOT-23" H 4950 4400 50  0001 C CNN
 F 3 "https://www.diodes.com/assets/Datasheets/AP7333.pdf" H 5150 4500 50  0001 C CNN
 	1    4900 4050
@@
 F 0 "C4" H 5592 4196 50  0000 L CNN
 F 1 "1uF" H 5592 4105 50  0000 L CNN
-F 2 "" H 5500 4150 50  0001 C CNN
+F 2 "Capacitor_SMD:C_0603_1608Metric" H 5500 4150 50  0001 C CNN
 F 3 "~" H 5500 4150 50  0001 C CNN
 	1    5500 4150
@@
 F 0 "C1" H 4392 4196 50  0000 L CNN
 F 1 "1uF" H 4392 4105 50  0000 L CNN
-F 2 "" H 4300 4150 50  0001 C CNN
+F 2 "Capacitor_SMD:C_0603_1608Metric" H 4300 4150 50  0001 C CNN
 F 3 "~" H 4300 4150 50  0001 C CNN
 	1    4300 4150
@@
 F 0 "U3" H 4900 5842 50  0000 C CNN
 F 1 "AP7333-15SRG-7" H 4900 5751 50  0000 C CNN
-F 2 "TO_SOT_Packages_SMD:SOT-23" H 4950 5900 50  0001 C CNN
+F 2 "Package_TO_SOT_SMD:SOT-23" H 4950 5900 50  0001 C CNN
 F 3 "https://www.diodes.com/assets/Datasheets/AP7333.pdf" H 5150 6000 50  0001 C CNN
 	1    4900 5550
@@
 F 0 "C5" H 5592 5696 50  0000 L CNN
 F 1 "1uF" H 5592 5605 50  0000 L CNN
-F 2 "" H 5500 5650 50  0001 C CNN
+F 2 "Capacitor_SMD:C_0603_1608Metric" H 5500 5650 50  0001 C CNN
 F 3 "~" H 5500 5650 50  0001 C CNN
 	1    5500 5650
@@
 F 0 "C2" H 4392 5696 50  0000 L CNN
 F 1 "1uF" H 4392 5605 50  0000 L CNN
-F 2 "" H 4300 5650 50  0001 C CNN
+F 2 "Capacitor_SMD:C_0603_1608Metric" H 4300 5650 50  0001 C CNN
 F 3 "~" H 4300 5650 50  0001 C CNN
 	1    4300 5650
@@
 F 0 "C3" V 5171 1100 50  0000 C CNN
 F 1 "1uF" V 5262 1100 50  0000 C CNN
-F 2 "" H 5400 1100 50  0001 C CNN
+F 2 "Capacitor_SMD:C_0603_1608Metric" H 5400 1100 50  0001 C CNN
 F 3 "~" H 5400 1100 50  0001 C CNN
 	1    5400 1100
@@
 F 0 "R1" H 5959 1996 50  0000 L CNN
 F 1 "4K7" H 5959 1905 50  0000 L CNN
-F 2 "" H 5900 1950 50  0001 C CNN
+F 2 "Resistor_SMD:R_0603_1608Metric" H 5900 1950 50  0001 C CNN
 F 3 "~" H 5900 1950 50  0001 C CNN
 	1    5900 1950
@@
 F 0 "R2" H 5959 2896 50  0000 L CNN
 F 1 "4K7" H 5959 2805 50  0000 L CNN
-F 2 "" H 5900 2850 50  0001 C CNN
+F 2 "Resistor_SMD:R_0603_1608Metric" H 5900 2850 50  0001 C CNN
 F 3 "~" H 5900 2850 50  0001 C CNN
 	1    5900 2850
@@
 Input Ports \n
 $Comp
-L Connector_Generic:Conn_01x10 J?
+L Connector_Generic:Conn_01x10 J4
 U 1 1 5C4EF787
 P 3750 6850
-F 0 "J?" H 3830 6842 50  0000 L CNN
+F 0 "J4" H 3830 6842 50  0000 L CNN
 F 1 "Conn_01x10" H 3830 6751 50  0000 L CNN
-F 2 "" H 3750 6850 50  0001 C CNN
+F 2 "Connector_PinHeader_2.54mm:PinHeader_1x10_P2.54mm_Vertical" H 3750 6850 50  0001 C CNN
 F 3 "~" H 3750 6850 50  0001 C CNN
 	1    3750 6850
 	1    0    0    -1
 $EndComp
+$Comp
+L power:+3V3 #PWR037
+U 1 1 5C31F193
+P 3150 6450
+F 0 "#PWR037" H 3150 6300 50  0001 C CNN
+F 1 "+3V3" H 3150 6600 50  0000 C CNN
+F 2 "" H 3150 6450 50  0001 C CNN
+F 3 "" H 3150 6450 50  0001 C CNN
+	1    3150 6450
+	1    0    0    -1
+$EndComp
+$Comp
+L power:+1V5 #PWR036
+U 1 1 5C31F1FE
+P 2950 6600
+F 0 "#PWR036" H 2950 6450 50  0001 C CNN
+F 1 "+1V5" H 2965 6773 50  0000 C CNN
+F 2 "" H 2950 6600 50  0001 C CNN
+F 3 "" H 2950 6600 50  0001 C CNN
+	1    2950 6600
+	1    0    0    -1
+$EndComp
+$Comp
+L power:+5V #PWR039
+U 1 1 5C31F239
+P 3300 6350
+F 0 "#PWR039" H 3300 6200 50  0001 C CNN
+F 1 "+5V" H 3315 6523 50  0000 C CNN
+F 2 "" H 3300 6350 50  0001 C CNN
+F 3 "" H 3300 6350 50  0001 C CNN
+	1    3300 6350
+	1    0    0    -1
+$EndComp
+Text Label 6250 4800 2    50   ~ 0
+SELECT
+Wire Wire Line
+	6250 4800 6500 4800
+Wire Wire Line
+	6500 4800 6500 4600
+Wire Wire Line
+	6500 4800 6500 5000
+Connection ~ 6500 4800
+$Comp
+L Device:R_Small R3
+U 1 1 5C33605B
+P 6500 4500
+F 0 "R3" H 6559 4546 50  0000 L CNN
+F 1 "1K8" H 6559 4455 50  0000 L CNN
+F 2 "Resistor_SMD:R_0603_1608Metric" H 6500 4500 50  0001 C CNN
+F 3 "~" H 6500 4500 50  0001 C CNN
+	1    6500 4500
+	1    0    0    -1
+$EndComp
+$Comp
+L Device:R_Small R4
+U 1 1 5C33624B
+P 6500 5100
+F 0 "R4" H 6559 5146 50  0000 L CNN
+F 1 "1K5" H 6559 5055 50  0000 L CNN
+F 2 "Resistor_SMD:R_0603_1608Metric" H 6500 5100 50  0001 C CNN
+F 3 "~" H 6500 5100 50  0001 C CNN
+	1    6500 5100
+	1    0    0    -1
+$EndComp
+Wire Wire Line
+	6500 4400 6500 4200
+$Comp
+L power:+3V3 #PWR040
+U 1 1 5C341AC3
+P 6500 4200
+F 0 "#PWR040" H 6500 4050 50  0001 C CNN
+F 1 "+3V3" H 6515 4373 50  0000 C CNN
+F 2 "" H 6500 4200 50  0001 C CNN
+F 3 "" H 6500 4200 50  0001 C CNN
+	1    6500 4200
+	1    0    0    -1
+$EndComp
+Wire Wire Line
+	3300 6350 3300 6450
+Wire Wire Line
+	3300 6450 3550 6450
+Wire Wire Line
+	3150 6450 3150 6550
+Wire Wire Line
+	3150 6550 3550 6550
+Wire Wire Line
+	2950 6600 2950 6650
+Wire Wire Line
+	2950 6650 3550 6650
+Wire Wire Line
+	3550 7350 3150 7350
+Wire Wire Line
+	3150 7350 3150 7550
+$Comp
+L power:GND #PWR038
+U 1 1 5C3724FE
+P 3150 7550
+F 0 "#PWR038" H 3150 7300 50  0001 C CNN
+F 1 "GND" H 3155 7377 50  0000 C CNN
+F 2 "" H 3150 7550 50  0001 C CNN
+F 3 "" H 3150 7550 50  0001 C CNN
+	1    3150 7550
+	1    0    0    -1
+$EndComp
+Wire Wire Line
+	3550 6750 3300 6750
+Wire Wire Line
+	3550 6850 3300 6850
+Wire Wire Line
+	3550 6950 3300 6950
+Wire Wire Line
+	3550 7050 3300 7050
+Wire Wire Line
+	3550 7150 3300 7150
+Wire Wire Line
+	3550 7250 3300 7250
+Text Label 3300 6850 2    50   ~ 0
+OUTCEC
+Text Label 3300 7050 2    50   ~ 0
+OUTSCL
+Text Label 3300 7150 2    50   ~ 0
+OUTUTIL
+Text Label 3300 7250 2    50   ~ 0
+OUTHBD
+Text Label 3300 6950 2    50   ~ 0
+OUTSDA
+Text Label 3300 6750 2    50   ~ 0
+OUTSEL
+Text Label 6750 5350 0    50   ~ 0
+OUTSEL
+Wire Wire Line
+	6500 5200 6500 5350
+Wire Wire Line
+	6500 5350 6750 5350
 $EndSCHEMATC

Commit message: differential traces done on hdmy
Parts:
- J1, J2, J3: footprint Connector_HDMI:HDMI_A_Contact_Technology_HDMI-19APL2_Horizontal -> digikey-footprints:HDMI_A_Female_2000-1-2-41-00-BK
Changed lines of the file:
@@
 F 0 "J1" H 2180 5596 50  0000 L CNN
 F 1 "HDMI_A" H 2180 5505 50  0000 L CNN
-F 2 "Connector_HDMI:HDMI_A_Contact_Technology_HDMI-19APL2_Horizontal" H 1775 5550 50  0001 C CNN
+F 2 "digikey-footprints:HDMI_A_Female_2000-1-2-41-00-BK" H 1775 5550 50  0001 C CNN
 F 3 "https://en.wikipedia.org/wiki/HDMI" H 1775 5550 50  0001 C CNN
 	1    1750 5550
@@
 F 0 "J3" H 10630 3346 50  0000 L CNN
 F 1 "HDMI_A" H 10630 3255 50  0000 L CNN
-F 2 "Connector_HDMI:HDMI_A_Contact_Technology_HDMI-19APL2_Horizontal" H 10225 3300 50  0001 C CNN
+F 2 "digikey-footprints:HDMI_A_Female_2000-1-2-41-00-BK" H 10225 3300 50  0001 C CNN
 F 3 "https://en.wikipedia.org/wiki/HDMI" H 10225 3300 50  0001 C CNN
 	1    10200 3300
@@
 F 0 "J2" H 8580 3346 50  0000 L CNN
 F 1 "HDMI_A" H 8580 3255 50  0000 L CNN
-F 2 "Connector_HDMI:HDMI_A_Contact_Technology_HDMI-19APL2_Horizontal" H 8175 3300 50  0001 C CNN
+F 2 "digikey-footprints:HDMI_A_Female_2000-1-2-41-00-BK" H 8175 3300 50  0001 C CNN
 F 3 "https://en.wikipedia.org/wiki/HDMI" H 8175 3300 50  0001 C CNN
 	1    8150 3300
